Commit message: Shifted traction to middle wheels

File: urdf/gazebo.xacro (robot description, xacro)
@@ -4,15 +4,43 @@
   <static>false</static>
 </gazebo>
+<gazebo reference="back_left_wheel_joint">
+  <mu1 value="${trolley_wheel_friction}"/>
+  <mu2 value="${trolley_wheel_friction}"/>
+  <kp  value="10000000.0" />
+  <kd  value="1.0" />
+  <fdir1 value="1 0 0"/>
+</gazebo>
+<gazebo reference="back_right_wheel_joint">
+  <mu1 value="${trolley_wheel_friction}"/>
+  <mu2 value="${trolley_wheel_friction}"/>
+  <kp  value="10000000.0" />
+  <kd  value="1.0" />
+  <fdir1 value="1 0 0"/>
+</gazebo>
+<gazebo reference="front_left_wheel_joint">
+  <mu1 value="${trolley_wheel_friction}"/>
+  <mu2 value="${trolley_wheel_friction}"/>
+  <kp  value="10000000.0" />
+  <kd  value="1.0" />
+  <fdir1 value="1 0 0"/>
+</gazebo>
+<gazebo reference="front_right_wheel_joint">
+  <mu1 value="${trolley_wheel_friction}"/>
+  <mu2 value="${trolley_wheel_friction}"/>
+  <kp  value="10000000.0" />
+  <kd  value="1.0" />
+  <fdir1 value="1 0 0"/>
+</gazebo>
 <!-- .....................MULTI WHEEL DIFF DRIVE ................................... -->
 <gazebo>
-	<plugin name="diffdrive_plugin_multiwheel" filename="libdiffdrive_plugin_multi_wheel.so">
+	<plugin name="diffdrive_plugin_multiwheel_middle" filename="libdiffdrive_plugin_multi_wheel.so">
 		<robotNamespace></robotNamespace>
 		<updateRate>100.0</updateRate>
-		<leftJoints>back_left_wheel_joint front_left_wheel_joint</leftJoints>
-		<rightJoints>back_right_wheel_joint front_right_wheel_joint</rightJoints>
-		<wheelSeparation>${wheel_base}</wheelSeparation>
+		<leftJoints>middle_left_wheel_joint</leftJoints>
+		<rightJoints>middle_right_wheel_joint</rightJoints>
+		<wheelSeparation>${traction_wheel_base}</wheelSeparation>
 		<wheelDiameter>${2*wheel_radius}</wheelDiameter>
 		<robotBaseFrame>base_link</robotBaseFrame>
-		<torque>${wheel_torque}</torque>
+		<torque>${traction_wheel_torque}</torque>
 		<commandTopic>/cmd_vel</commandTopic>
 		<odometryTopic>odom</odometryTopic>
@@ -22,20 +50,4 @@
 	</plugin>
 </gazebo>
-<gazebo>
-	<plugin name="diffdrive_plugin_multiwheel_middle" filename="libdiffdrive_plugin_multi_wheel.so">
-		<robotNamespace></robotNamespace>
-		<updateRate>100.0</updateRate>
-		<leftJoints>middle_left_wheel_joint</leftJoints>
-		<rightJoints>middle_right_wheel_joint</rightJoints>
-		<wheelSeparation>${wheel_middle_base}</wheelSeparation>
-		<wheelDiameter>${2*wheel_radius}</wheelDiameter>
-		<robotBaseFrame>base_link</robotBaseFrame>
-		<torque>${wheel_torque}</torque>
-		<commandTopic>/cmd_vel</commandTopic>
-		<odometryTopic>odom</odometryTopic>
-		<odometryFrame>odom</odometryFrame>
-		<publishOdometryTf>true</publishOdometryTf>
-		<publishOdometryMsg>true</publishOdometryMsg>
-	</plugin>
-</gazebo>
+<!--................................................................................. -->
 </robot>

File: urdf/macros.xacro (robot description, xacro)
@@ -38,6 +38,12 @@
     <inertial>
       <origin xyz="0 0 0" rpy="0 ${pi/2} ${pi/2}" />
-      <mass value="${wheel_mass}"/>
-      <xacro:cylinder_inertia m="${wheel_mass}" r="${wheel_radius}" h="${wheel_width}"/>
+    <xacro:if value="${cardinality == 'middle'}">
+        <mass value="${traction_wheel_mass}"/>
+				<xacro:cylinder_inertia m="${traction_wheel_mass}" r="${wheel_radius}" h="${wheel_width}"/>
+    </xacro:if>
+    <xacro:unless value="${cardinality == 'middle'}">
+        <mass value="${trolley_wheel_mass}"/>
+				<xacro:cylinder_inertia m="${trolley_wheel_mass}" r="${wheel_radius}" h="${wheel_width}"/>
+    </xacro:unless>
     </inertial>
    </link>

File: urdf/new_bcr_robot.xacro (robot description, xacro)
@@ -2,10 +2,13 @@
 <robot xmlns:xacro="http://www.ros.org/wiki/xacro" name="new_bcr_robot">
 <!--................................ XACRO CONSTANTS .............................. -->
-<xacro:property name="wheel_mass"                           value="1"/>
+<xacro:property name="chassis_mass"                    				value="0.1"/>
+<xacro:property name="traction_wheel_mass"                    value="1"/>
+<xacro:property name="traction_wheel_base"                    value="0.44"/>
+<xacro:property name="traction_wheel_torque"                  value="50"/>
+<xacro:property name="trolley_wheel_mass"                    	value="0.1"/>
+<xacro:property name="trolley_wheel_base"                  		value="0.54"/>
+<xacro:property name="trolley_wheel_friction"               	value="1.0"/>
 <xacro:property name="wheel_radius"                         value="0.06"/>
 <xacro:property name="wheel_width"                          value="0.025"/>
-<xacro:property name="wheel_middle_base"                    value="0.44"/>
-<xacro:property name="wheel_base"                  					value="0.54"/>
-<xacro:property name="wheel_torque"                         value="10"/>
 <!-- ............................... LOAD MACROS ................................. -->
 <xacro:include filename="$(find new_bcr_robot)/urdf/materials.xacro"/>
@@ -23,14 +26,14 @@
 	</visual>
 	<inertial>
-		<mass value="1"/>
+		<mass value="${chassis_mass}" />
 		<inertia ixx="0.01" ixy="0" ixz="0" iyy="0.01" iyz="0" izz="0.01"/>
 	</inertial>
 </link>
 <!-- ................................ WHEELS ..................................... -->
-<xacro:wheel cardinality="front" dexterity="left"  origin_x="0.37" origin_y="${wheel_base/2}" origin_z="${wheel_radius}"/>
-<xacro:wheel cardinality="front" dexterity="right" origin_x="0.37" origin_y="-${wheel_base/2}" origin_z="${wheel_radius}"/>
-<xacro:wheel cardinality="back" dexterity="left"  origin_x="-0.37" origin_y="${wheel_base/2}" origin_z="${wheel_radius}"/>
-<xacro:wheel cardinality="back" dexterity="right" origin_x="-0.37" origin_y="-${wheel_base/2}" origin_z="${wheel_radius}"/>
-<xacro:wheel cardinality="middle" dexterity="left"  origin_x="0" origin_y="${wheel_middle_base/2}" origin_z="${wheel_radius}"/>
-<xacro:wheel cardinality="middle" dexterity="right" origin_x="0" origin_y="-${wheel_middle_base/2}" origin_z="${wheel_radius}"/>
+<xacro:wheel cardinality="front" dexterity="left"  origin_x="0.37" origin_y="${trolley_wheel_base/2}" origin_z="${wheel_radius}"/>
+<xacro:wheel cardinality="front" dexterity="right" origin_x="0.37" origin_y="-${trolley_wheel_base/2}" origin_z="${wheel_radius}"/>
+<xacro:wheel cardinality="back" dexterity="left"  origin_x="-0.37" origin_y="${trolley_wheel_base/2}" origin_z="${wheel_radius}"/>
+<xacro:wheel cardinality="back" dexterity="right" origin_x="-0.37" origin_y="-${trolley_wheel_base/2}" origin_z="${wheel_radius}"/>
+<xacro:wheel cardinality="middle" dexterity="left"  origin_x="0" origin_y="${traction_wheel_base/2}" origin_z="${wheel_radius}"/>
+<xacro:wheel cardinality="middle" dexterity="right" origin_x="0" origin_y="-${traction_wheel_base/2}" origin_z="${wheel_radius}"/>
 </robot>

Commit message: Added LiDAR and IMU

File: urdf/gazebo.xacro (robot description, xacro)
@@ -50,4 +50,65 @@
 	</plugin>
 </gazebo>
+<!--............................... IMU PLUGIN ..................................... -->
+<gazebo>
+	<plugin name="imu_plugin" filename="libgazebo_ros_imu.so">
+			<updateRate>50.0</updateRate>
+			<bodyName>base_link</bodyName>
+			<topicName>/imu</topicName>
+			<serviceName>/imu/calibrate</serviceName>
+			<accelOffset>0.0 0.0 0.0</accelOffset>
+			<accelDrift>0.0 0.0 0.0</accelDrift>
+			<accelDriftFrequency>0.0 0.0 0.0</accelDriftFrequency>
+			<accelGaussianNoise>0.0 0.0 0.0</accelGaussianNoise>
+			<rateOffset>0.0 0.0 0.0</rateOffset>
+			<rateDrift>0.0 0.0 0.0</rateDrift>
+			<rateDriftFrequency>0.0 0.0 0.0</rateDriftFrequency>
+			<rateGaussianNoise>0.0 0.0 0.0</rateGaussianNoise>
+			<headingOffset>0.0</headingOffset>
+			<headingDrift>0.0</headingDrift>
+			<headingDriftFrequency>0.0</headingDriftFrequency>
+			<headingGaussianNoise>0.0</headingGaussianNoise>
+			<rpyOffset>0.0 0.0 0.0</rpyOffset>
+			<xyzOffset>0.0 0.0 0.0</xyzOffset>
+			<gaussianNoise>0.0</gaussianNoise>
+			<frameName>imu_frame</frameName>
+	</plugin>
+</gazebo>
+<!-- ........................... 2D LIDAR PLUGIN ................................... -->
+<xacro:if value="$(arg two_d_lidar_enabled)">
+   <gazebo reference="two_d_lidar">
+      <gravity>true</gravity>
+      <sensor type="ray" name="two_d_lidar">
+        <pose>0 0 0 0 0 0</pose>
+        <visualize>false</visualize>
+        <update_rate>${two_d_lidar_update_rate}</update_rate>
+        <ray>
+          <scan>
+            <horizontal>
+              <samples>${two_d_lidar_sample_size}</samples>
+              <resolution>1</resolution>
+              <min_angle>${radians(two_d_lidar_min_angle)}</min_angle>
+              <max_angle>${radians(two_d_lidar_max_angle)}</max_angle>
+            </horizontal>
+          </scan>
+          <range>
+            <min>${two_d_lidar_min_range}</min>
+            <max>${two_d_lidar_max_range}</max>
+            <resolution>0.01</resolution>
+          </range>
+          <noise>
+            <type>gaussian</type>
+            <mean>0.0</mean>
+            <stddev>0.001</stddev>
+          </noise>
+        </ray>
+        <plugin name="gazebo_ros_laser" filename="libgazebo_ros_laser.so">
+          <topicName>scan</topicName>
+          <frameName>two_d_lidar</frameName>
+          <robotNamespace>/</robotNamespace>
+        </plugin>
+      </sensor>
+   </gazebo>
+</xacro:if>
 <!--................................................................................. -->
 </robot>

File: urdf/new_bcr_robot.xacro (robot description, xacro)
@@ -11,4 +11,11 @@
 <xacro:property name="wheel_radius"                         value="0.06"/>
 <xacro:property name="wheel_width"                          value="0.025"/>
+<xacro:arg      name="two_d_lidar_enabled"                  default="true" />
+<xacro:property name="two_d_lidar_update_rate"              value="50"/>
+<xacro:property name="two_d_lidar_sample_size"              value="361"/>
+<xacro:property name="two_d_lidar_min_angle"                value="0"/>
+<xacro:property name="two_d_lidar_max_angle"                value="360"/>
+<xacro:property name="two_d_lidar_min_range"                value="0.1"/>
+<xacro:property name="two_d_lidar_max_range"                value="16"/>
 <!-- ............................... LOAD MACROS ................................. -->
 <xacro:include filename="$(find new_bcr_robot)/urdf/materials.xacro"/>
@@ -37,3 +44,34 @@
 <xacro:wheel cardinality="middle" dexterity="left"  origin_x="0" origin_y="${traction_wheel_base/2}" origin_z="${wheel_radius}"/>
 <xacro:wheel cardinality="middle" dexterity="right" origin_x="0" origin_y="-${traction_wheel_base/2}" origin_z="${wheel_radius}"/>
+<!-- ............................. 2D LIDAR ........................................ -->
+<xacro:if value="$(arg two_d_lidar_enabled)">
+    <link name="two_d_lidar">
+        <collision>
+          <origin xyz="0 0 0" rpy="0 0 0" />
+          <geometry>
+           <cylinder length="0.06" radius="0.075"/>
+          </geometry>
+        </collision>
+        <visual>
+          <origin xyz="0 0 0" rpy="0 0 0" />
+          <geometry>
+           <cylinder length="0.06" radius="0.075"/>
+          </geometry>
+          <material name="orange"/>
+        </visual>
+        <inertial>
+          <origin xyz="0 0 0" rpy="0 0 0" />
+          <mass value="0.1"/>
+          <xacro:cylinder_inertia m="0.1" r="0.075" h="0.06"/>
+        </inertial>
+   </link>
+   <joint name="two_d_lidar_joint" type="fixed">
+      <parent link="base_link"/>
+      <child link="two_d_lidar"/>
+      <origin xyz="0.3 0 0.45" rpy="0 0 ${-pi/2}" />
+    </joint>
+   <gazebo reference="two_d_lidar">
+       <material>Gazebo/Orange</material>
+   </gazebo>
+</xacro:if>
 </robot>

Commit message: Added collision

File: urdf/gazebo.xacro (robot description, xacro)
@@ -28,4 +28,18 @@
   <mu1 value="${trolley_wheel_friction}"/>
   <mu2 value="${trolley_wheel_friction}"/>
+  <kp  value="10000000.0" />
+  <kd  value="1.0" />
+  <fdir1 value="1 0 0"/>
+</gazebo>
+<gazebo reference="middle_left_wheel_joint">
+  <mu1 value="${traction_wheel_friction}"/>
+  <mu2 value="${traction_wheel_friction}"/>
+  <kp  value="10000000.0" />
+  <kd  value="1.0" />
+  <fdir1 value="1 0 0"/>
+</gazebo>
+<gazebo reference="middle_right_wheel_joint">
+  <mu1 value="${traction_wheel_friction}"/>
+  <mu2 value="${traction_wheel_friction}"/>
   <kp  value="10000000.0" />
   <kd  value="1.0" />

File: urdf/new_bcr_robot.xacro (robot description, xacro)
@@ -2,13 +2,19 @@
 <robot xmlns:xacro="http://www.ros.org/wiki/xacro" name="new_bcr_robot">
 <!--................................ XACRO CONSTANTS .............................. -->
-<xacro:property name="chassis_mass"                    				value="0.1"/>
-<xacro:property name="traction_wheel_mass"                    value="1"/>
-<xacro:property name="traction_wheel_base"                    value="0.44"/>
-<xacro:property name="traction_wheel_torque"                  value="50"/>
-<xacro:property name="trolley_wheel_mass"                    	value="0.1"/>
-<xacro:property name="trolley_wheel_base"                  		value="0.54"/>
-<xacro:property name="trolley_wheel_friction"               	value="1.0"/>
+<xacro:property name="chassis_mass"                    			value="0.1"/>
+<xacro:property name="chassis_length"                    		value="0.95"/>
+<xacro:property name="chassis_width"                    		value="0.64"/>
+<xacro:property name="chassis_height"                    		value="0.25"/>
+<xacro:property name="chassis_ground_clearance"             value="0.16"/>
+<xacro:property name="traction_wheel_mass"                  value="1"/>
+<xacro:property name="traction_wheel_base"                  value="0.44"/>
+<xacro:property name="traction_wheel_torque"                value="50"/>
+<xacro:property name="traction_wheel_friction"              value="5.0"/>
+<xacro:property name="trolley_wheel_mass"                   value="0.1"/>
+<xacro:property name="trolley_wheel_base"                  	value="0.54"/>
+<xacro:property name="trolley_wheel_friction"               value="0.0"/>
 <xacro:property name="wheel_radius"                         value="0.06"/>
 <xacro:property name="wheel_width"                          value="0.025"/>
+<xacro:property name="wheel_pos"                          	value="0.37"/>
 <xacro:arg      name="two_d_lidar_enabled"                  default="true" />
 <xacro:property name="two_d_lidar_update_rate"              value="50"/>
@@ -22,24 +28,28 @@
 <xacro:include filename="$(find new_bcr_robot)/urdf/macros.xacro"/>
 <xacro:include filename="$(find new_bcr_robot)/urdf/gazebo.xacro"/>
-<!--.............................................................................. -->
 <!-- ................................ BASE LINK .................................. -->
 <link name="base_link">
+	<collision>
+		<origin xyz="0 0 ${chassis_ground_clearance + chassis_height/2}" rpy="0 0 0" />
+  		<geometry>
+				<box size="${chassis_length} ${chassis_width} ${chassis_height}"/>
+  		</geometry>
+	</collision>
 	<visual>
-		<origin xyz="0 0 0.16" rpy="0 0 0" />
+		<origin xyz="0 0 ${chassis_ground_clearance}" rpy="0 0 0" />
   		<geometry>
     		<mesh filename="package://new_bcr_robot/meshes/bcr_chassis.dae" scale="0.1 0.1 0.1"/>
-				<scale>0.01 0.01 0.01</scale>
   		</geometry>
 	</visual>
 	<inertial>
 		<mass value="${chassis_mass}" />
-		<inertia ixx="0.01" ixy="0" ixz="0" iyy="0.01" iyz="0" izz="0.01"/>
+		<xacro:box_inertia m="${chassis_mass}" x="${chassis_length}" y="${chassis_width}" z = "${chassis_height}"/>
 	</inertial>
 </link>
 <!-- ................................ WHEELS ..................................... -->
-<xacro:wheel cardinality="front" dexterity="left"  origin_x="0.37" origin_y="${trolley_wheel_base/2}" origin_z="${wheel_radius}"/>
-<xacro:wheel cardinality="front" dexterity="right" origin_x="0.37" origin_y="-${trolley_wheel_base/2}" origin_z="${wheel_radius}"/>
-<xacro:wheel cardinality="back" dexterity="left"  origin_x="-0.37" origin_y="${trolley_wheel_base/2}" origin_z="${wheel_radius}"/>
-<xacro:wheel cardinality="back" dexterity="right" origin_x="-0.37" origin_y="-${trolley_wheel_base/2}" origin_z="${wheel_radius}"/>
+<xacro:wheel cardinality="front" dexterity="left"  origin_x="${wheel_pos}" origin_y="${trolley_wheel_base/2}" origin_z="${wheel_radius}"/>
+<xacro:wheel cardinality="front" dexterity="right" origin_x="${wheel_pos}" origin_y="-${trolley_wheel_base/2}" origin_z="${wheel_radius}"/>
+<xacro:wheel cardinality="back" dexterity="left"  origin_x="-${wheel_pos}" origin_y="${trolley_wheel_base/2}" origin_z="${wheel_radius}"/>
+<xacro:wheel cardinality="back" dexterity="right" origin_x="-${wheel_pos}" origin_y="-${trolley_wheel_base/2}" origin_z="${wheel_radius}"/>
 <xacro:wheel cardinality="middle" dexterity="left"  origin_x="0" origin_y="${traction_wheel_base/2}" origin_z="${wheel_radius}"/>
 <xacro:wheel cardinality="middle" dexterity="right" origin_x="0" origin_y="-${traction_wheel_base/2}" origin_z="${wheel_radius}"/>
