Commit message: changes in modelling, improved velocity response

File: urdf/gazebo.xacro (robot description, xacro)
@@ -48,18 +48,20 @@
 <!-- .....................MULTI WHEEL DIFF DRIVE ................................... -->
 <gazebo>
-	<plugin name="diffdrive_plugin_multiwheel_middle" filename="libdiffdrive_plugin_multi_wheel.so">
+	<plugin name="diffdrive_plugin_multiwheel_middle" filename="libgazebo_ros_diff_drive.so">
 		<robotNamespace></robotNamespace>
+    <legacyMode>false</legacyMode>
 		<updateRate>100.0</updateRate>
-		<leftJoints>middle_left_wheel_joint</leftJoints>
-		<rightJoints>middle_right_wheel_joint</rightJoints>
-		<wheelSeparation>${traction_wheel_base}</wheelSeparation>
-		<wheelDiameter>${2*wheel_radius}</wheelDiameter>
+		<leftJoint>middle_left_wheel_joint</leftJoint>
+		<rightJoint>middle_right_wheel_joint</rightJoint>
+		<wheelSeparation>${traction_wheel_base+traction_wheel_width}</wheelSeparation>
+		<wheelDiameter>${2*traction_wheel_radius}</wheelDiameter>
 		<robotBaseFrame>base_link</robotBaseFrame>
-		<torque>${traction_wheel_torque}</torque>
+		<wheelTorque>${traction_wheel_torque}</wheelTorque>
 		<commandTopic>/cmd_vel</commandTopic>
-		<odometryTopic>odom</odometryTopic>
+		<odometryTopic>/odom</odometryTopic>
 		<odometryFrame>odom</odometryFrame>
 		<publishOdometryTf>true</publishOdometryTf>
 		<publishOdometryMsg>true</publishOdometryMsg>
+    <wheelAcceleration>5.0</wheelAcceleration>
 	</plugin>
 </gazebo>

File: urdf/macros.xacro (robot description, xacro)
@@ -20,11 +20,11 @@
     />
   </xacro:macro>
-<!-- ............................... WHEEL DEFINITION .............................. -->
- <xacro:macro name="wheel" params="cardinality dexterity origin_x origin_y origin_z">
+<!-- ............................... TROLLEY WHEEL DEFINITION .............................. -->
+ <xacro:macro name="trolley_wheel" params="cardinality dexterity origin_x origin_y origin_z">
    <link name="${cardinality}_${dexterity}_wheel">
     <collision>
       <origin xyz="0 0 0" rpy="0 ${pi/2} ${pi/2}" />
       <geometry>
-       <cylinder length="${wheel_width}" radius="${wheel_radius}"/>
+       <sphere radius="${trolley_wheel_radius}"/>
       </geometry>
     </collision>
@@ -32,5 +32,37 @@
       <origin xyz="0 0 0" rpy="0 ${pi/2} ${pi/2}" />
       <geometry>
-       <cylinder length="${wheel_width}" radius="${wheel_radius}"/>
+       <sphere radius="${trolley_wheel_radius}"/>
+      </geometry>
+      <material name="black"/>
+    </visual>
+    <inertial>
+      <origin xyz="0 0 0" rpy="0 0 0" />
+      <mass value="${trolley_wheel_mass}"/>
+				<xacro:sphere_inertia m="${trolley_wheel_mass}" r="${trolley_wheel_radius}"/>
+    </inertial>
+    <mu>0.0</mu>
+   </link>
+   <joint name="${cardinality}_${dexterity}_wheel_joint" type="fixed">
+      <parent link="base_link"/>
+      <child link="${cardinality}_${dexterity}_wheel"/>
+      <origin xyz="${origin_x} ${origin_y} ${origin_z}" rpy="0 0 0" />
+      <axis xyz="0 1 0" rpy="0 0 0" />
+    </joint>
+   <gazebo reference="${cardinality}_${dexterity}_wheel">
+      <material>Gazebo/Black</material>
+   </gazebo>
+  </xacro:macro>
+ <xacro:macro name="traction_wheel" params="cardinality dexterity origin_x origin_y origin_z">
+   <link name="${cardinality}_${dexterity}_wheel">
+    <collision>
+      <origin xyz="0 0 0" rpy="0 ${pi/2} ${pi/2}" />
+      <geometry>
+       <cylinder length="${traction_wheel_width}" radius="${traction_wheel_radius}"/>
+      </geometry>
+    </collision>
+    <visual>
+      <origin xyz="0 0 0" rpy="0 ${pi/2} ${pi/2}" />
+      <geometry>
+       <cylinder length="${traction_wheel_width}" radius="${traction_wheel_radius}"/>
       </geometry>
       <material name="black"/>
@@ -38,13 +70,8 @@
     <inertial>
       <origin xyz="0 0 0" rpy="0 ${pi/2} ${pi/2}" />
-    <xacro:if value="${cardinality == 'middle'}">
-        <mass value="${traction_wheel_mass}"/>
-				<xacro:cylinder_inertia m="${traction_wheel_mass}" r="${wheel_radius}" h="${wheel_width}"/>
-    </xacro:if>
-    <xacro:unless value="${cardinality == 'middle'}">
-        <mass value="${trolley_wheel_mass}"/>
-				<xacro:cylinder_inertia m="${trolley_wheel_mass}" r="${wheel_radius}" h="${wheel_width}"/>
-    </xacro:unless>
+      <mass value="${traction_wheel_mass}"/>
+      <xacro:cylinder_inertia m="${traction_wheel_mass}" r="${traction_wheel_radius}" h="${traction_wheel_width}"/>
     </inertial>
+    <mu>5.0</mu>
    </link>
    <joint name="${cardinality}_${dexterity}_wheel_joint" type="continuous">

File: urdf/new_bcr_robot.xacro (robot description, xacro)
@@ -2,22 +2,25 @@
 <robot xmlns:xacro="http://www.ros.org/wiki/xacro" name="new_bcr_robot">
 <!--................................ XACRO CONSTANTS .............................. -->
-<xacro:property name="chassis_mass"                    			value="0.1"/>
-<xacro:property name="chassis_length"                    		value="0.95"/>
-<xacro:property name="chassis_width"                    		value="0.64"/>
-<xacro:property name="chassis_height"                    		value="0.25"/>
-<xacro:property name="chassis_ground_clearance"             value="0.16"/>
+<xacro:property name="chassis_mass"                    		value="70"/>
+<xacro:property name="chassis_length"                    	value="0.95"/>
+<xacro:property name="chassis_width"                    	value="0.64"/>
+<xacro:property name="chassis_height"                    	value="0.25"/>
+<xacro:property name="chassis_ground_clearance"             value="0.5"/>
 <xacro:property name="traction_wheel_mass"                  value="1"/>
-<xacro:property name="traction_wheel_base"                  value="0.44"/>
-<xacro:property name="traction_wheel_torque"                value="50"/>
+<xacro:property name="traction_wheel_base"                  value="0.88"/>
+<xacro:property name="traction_wheel_torque"                value="20000"/>
 <xacro:property name="traction_wheel_friction"              value="5.0"/>
 <xacro:property name="trolley_wheel_mass"                   value="0.1"/>
 <xacro:property name="trolley_wheel_base"                  	value="0.54"/>
 <xacro:property name="trolley_wheel_friction"               value="0.0"/>
-<xacro:property name="wheel_radius"                         value="0.06"/>
-<xacro:property name="wheel_width"                          value="0.025"/>
-<xacro:property name="wheel_pos"                          	value="0.37"/>
-<xacro:arg      name="two_d_lidar_enabled"                  default="true" />
-<xacro:property name="two_d_lidar_update_rate"              value="50"/>
-<xacro:property name="two_d_lidar_sample_size"              value="361"/>
+<xacro:property name="trolley_wheel_radius"                value="0.06"/>
+<!-- a small constant -->
+<xacro:property name="eps"                                  value="0.002"/>
+<xacro:property name="traction_wheel_radius"                value="0.1"/>
+<xacro:property name="traction_wheel_width"                          value="0.05"/>
+<xacro:property name="traction_wheel_base"                          	value="0.8"/>
+<xacro:arg      name="two_d_lidar_enabled"                  default="false" />
+<xacro:property name="two_d_lidar_update_rate"              value="30"/>
+<xacro:property name="two_d_lidar_sample_size"              value="720"/>
 <xacro:property name="two_d_lidar_min_angle"                value="0"/>
 <xacro:property name="two_d_lidar_max_angle"                value="360"/>
@@ -29,15 +32,16 @@
 <xacro:include filename="$(find new_bcr_robot)/urdf/gazebo.xacro"/>
 <!-- ................................ BASE LINK .................................. -->
+<link name="base_ref"/>
 <link name="base_link">
 	<collision>
-		<origin xyz="0 0 ${chassis_ground_clearance + chassis_height/2}" rpy="0 0 0" />
+		<origin xyz="0 0 0" rpy="0 0 0" />
   		<geometry>
-				<box size="${chassis_length} ${chassis_width} ${chassis_height}"/>
+			<box size="${chassis_length} ${chassis_width} ${chassis_height}"/>
   		</geometry>
 	</collision>
 	<visual>
-		<origin xyz="0 0 ${chassis_ground_clearance}" rpy="0 0 0" />
+		<origin xyz="0 0 0" rpy="0 0 0" />
   		<geometry>
-    		<mesh filename="package://new_bcr_robot/meshes/bcr_chassis.dae" scale="0.1 0.1 0.1"/>
+    		<box size="${chassis_length} ${chassis_width} ${chassis_height}"/>
   		</geometry>
 	</visual>
@@ -47,11 +51,16 @@
 	</inertial>
 </link>
+    <joint name="base_joint" type="fixed">
+      <parent link="base_ref"/>
+      <child link="base_link"/>
+      <origin xyz="0.0 0 0.0" rpy="0 0 0.0" />
+    </joint>
 <!-- ................................ WHEELS ..................................... -->
-<xacro:wheel cardinality="front" dexterity="left"  origin_x="${wheel_pos}" origin_y="${trolley_wheel_base/2}" origin_z="${wheel_radius}"/>
-<xacro:wheel cardinality="front" dexterity="right" origin_x="${wheel_pos}" origin_y="-${trolley_wheel_base/2}" origin_z="${wheel_radius}"/>
-<xacro:wheel cardinality="back" dexterity="left"  origin_x="-${wheel_pos}" origin_y="${trolley_wheel_base/2}" origin_z="${wheel_radius}"/>
-<xacro:wheel cardinality="back" dexterity="right" origin_x="-${wheel_pos}" origin_y="-${trolley_wheel_base/2}" origin_z="${wheel_radius}"/>
-<xacro:wheel cardinality="middle" dexterity="left"  origin_x="0" origin_y="${traction_wheel_base/2}" origin_z="${wheel_radius}"/>
-<xacro:wheel cardinality="middle" dexterity="right" origin_x="0" origin_y="-${traction_wheel_base/2}" origin_z="${wheel_radius}"/>
+<xacro:trolley_wheel cardinality="front" dexterity="left"  origin_x="${chassis_length/2}" origin_y="${trolley_wheel_base/2}" origin_z="-${trolley_wheel_radius+chassis_height/2}"/>
+<xacro:trolley_wheel cardinality="front" dexterity="right" origin_x="${chassis_length/2}" origin_y="-${trolley_wheel_base/2}" origin_z="-${trolley_wheel_radius+chassis_height/2}"/>
+<xacro:trolley_wheel cardinality="back" dexterity="left"  origin_x="-${chassis_length/2}" origin_y="${trolley_wheel_base/2}" origin_z="-${trolley_wheel_radius+chassis_height/2}"/>
+<xacro:trolley_wheel cardinality="back" dexterity="right" origin_x="-${chassis_length/2}" origin_y="-${trolley_wheel_base/2}" origin_z="-${trolley_wheel_radius+chassis_height/2}"/>
+<xacro:traction_wheel cardinality="middle" dexterity="left"  origin_x="0" origin_y="${traction_wheel_base/2}" origin_z="-${chassis_height/2+2*trolley_wheel_radius+eps-traction_wheel_radius}"/>
+<xacro:traction_wheel cardinality="middle" dexterity="right" origin_x="0" origin_y="-${traction_wheel_base/2}" origin_z="-${chassis_height/2+2*trolley_wheel_radius+eps-traction_wheel_radius}"/>
 <!-- ............................. 2D LIDAR ........................................ -->
 <xacro:if value="$(arg two_d_lidar_enabled)">

Commit message: Added visualization

File: urdf/gazebo.xacro (robot description, xacro)
@@ -3,46 +3,4 @@
 <gazebo>
   <static>false</static>
-</gazebo>
-<gazebo reference="back_left_wheel_joint">
-  <mu1 value="${trolley_wheel_friction}"/>
-  <mu2 value="${trolley_wheel_friction}"/>
-  <kp  value="10000000.0" />
-  <kd  value="1.0" />
-  <fdir1 value="1 0 0"/>
-</gazebo>
-<gazebo reference="back_right_wheel_joint">
-  <mu1 value="${trolley_wheel_friction}"/>
-  <mu2 value="${trolley_wheel_friction}"/>
-  <kp  value="10000000.0" />
-  <kd  value="1.0" />
-  <fdir1 value="1 0 0"/>
-</gazebo>
-<gazebo reference="front_left_wheel_joint">
-  <mu1 value="${trolley_wheel_friction}"/>
-  <mu2 value="${trolley_wheel_friction}"/>
-  <kp  value="10000000.0" />
-  <kd  value="1.0" />
-  <fdir1 value="1 0 0"/>
-</gazebo>
-<gazebo reference="front_right_wheel_joint">
-  <mu1 value="${trolley_wheel_friction}"/>
-  <mu2 value="${trolley_wheel_friction}"/>
-  <kp  value="10000000.0" />
-  <kd  value="1.0" />
-  <fdir1 value="1 0 0"/>
-</gazebo>
-<gazebo reference="middle_left_wheel_joint">
-  <mu1 value="${traction_wheel_friction}"/>
-  <mu2 value="${traction_wheel_friction}"/>
-  <kp  value="10000000.0" />
-  <kd  value="1.0" />
-  <fdir1 value="1 0 0"/>
-</gazebo>
-<gazebo reference="middle_right_wheel_joint">
-  <mu1 value="${traction_wheel_friction}"/>
-  <mu2 value="${traction_wheel_friction}"/>
-  <kp  value="10000000.0" />
-  <kd  value="1.0" />
-  <fdir1 value="1 0 0"/>
 </gazebo>
 <!-- .....................MULTI WHEEL DIFF DRIVE ................................... -->
@@ -61,6 +19,11 @@
 		<odometryTopic>/odom</odometryTopic>
 		<odometryFrame>odom</odometryFrame>
-		<publishOdometryTf>true</publishOdometryTf>
+		<rosDebugLevel>na</rosDebugLevel>
+		<publishTf>true</publishTf>
+		<publishOdomTF>true</publishOdomTF>
+		<publishWheelTF>false</publishWheelTF>
+		<publishWheelJointState>false</publishWheelJointState>
 		<publishOdometryMsg>true</publishOdometryMsg>
+		<odometrySource>world</odometrySource>
     <wheelAcceleration>5.0</wheelAcceleration>
 	</plugin>

File: urdf/macros.xacro (robot description, xacro)
@@ -29,11 +29,4 @@
       </geometry>
     </collision>
-    <visual>
-      <origin xyz="0 0 0" rpy="0 ${pi/2} ${pi/2}" />
-      <geometry>
-       <sphere radius="${trolley_wheel_radius}"/>
-      </geometry>
-      <material name="black"/>
-    </visual>
     <inertial>
       <origin xyz="0 0 0" rpy="0 0 0" />
@@ -61,11 +54,4 @@
       </geometry>
     </collision>
-    <visual>
-      <origin xyz="0 0 0" rpy="0 ${pi/2} ${pi/2}" />
-      <geometry>
-       <cylinder length="${traction_wheel_width}" radius="${traction_wheel_radius}"/>
-      </geometry>
-      <material name="black"/>
-    </visual>
     <inertial>
       <origin xyz="0 0 0" rpy="0 ${pi/2} ${pi/2}" />

File: urdf/new_bcr_robot.xacro (robot description, xacro)
@@ -6,25 +6,25 @@
 <xacro:property name="chassis_width"                    	value="0.64"/>
 <xacro:property name="chassis_height"                    	value="0.25"/>
-<xacro:property name="chassis_ground_clearance"             value="0.5"/>
-<xacro:property name="traction_wheel_mass"                  value="1"/>
-<xacro:property name="traction_wheel_base"                  value="0.88"/>
-<xacro:property name="traction_wheel_torque"                value="20000"/>
-<xacro:property name="traction_wheel_friction"              value="5.0"/>
-<xacro:property name="trolley_wheel_mass"                   value="0.1"/>
-<xacro:property name="trolley_wheel_base"                  	value="0.54"/>
-<xacro:property name="trolley_wheel_friction"               value="0.0"/>
-<xacro:property name="trolley_wheel_radius"                value="0.06"/>
+<xacro:property name="chassis_ground_clearance"           value="0.5"/>
+<xacro:property name="traction_wheel_mass"                value="1"/>
+<xacro:property name="traction_wheel_base"                value="0.88"/>
+<xacro:property name="traction_wheel_torque"              value="20000"/>
+<xacro:property name="traction_wheel_friction"            value="5.0"/>
+<xacro:property name="trolley_wheel_mass"                 value="0.1"/>
+<xacro:property name="trolley_wheel_base"                 value="0.54"/>
+<xacro:property name="trolley_wheel_friction"             value="0.0"/>
+<xacro:property name="trolley_wheel_radius"               value="0.06"/>
 <!-- a small constant -->
-<xacro:property name="eps"                                  value="0.002"/>
-<xacro:property name="traction_wheel_radius"                value="0.1"/>
-<xacro:property name="traction_wheel_width"                          value="0.05"/>
-<xacro:property name="traction_wheel_base"                          	value="0.8"/>
-<xacro:arg      name="two_d_lidar_enabled"                  default="false" />
-<xacro:property name="two_d_lidar_update_rate"              value="30"/>
-<xacro:property name="two_d_lidar_sample_size"              value="720"/>
-<xacro:property name="two_d_lidar_min_angle"                value="0"/>
-<xacro:property name="two_d_lidar_max_angle"                value="360"/>
-<xacro:property name="two_d_lidar_min_range"                value="0.1"/>
-<xacro:property name="two_d_lidar_max_range"                value="16"/>
+<xacro:property name="eps"                                value="0.002"/>
+<xacro:property name="traction_wheel_radius"              value="0.1"/>
+<xacro:property name="traction_wheel_width"               value="0.05"/>
+<xacro:property name="traction_wheel_base"                value="0.8"/>
+<xacro:arg      name="two_d_lidar_enabled"                default="false" />
+<xacro:property name="two_d_lidar_update_rate"            value="30"/>
+<xacro:property name="two_d_lidar_sample_size"            value="361"/>
+<xacro:property name="two_d_lidar_min_angle"              value="0"/>
+<xacro:property name="two_d_lidar_max_angle"              value="360"/>
+<xacro:property name="two_d_lidar_min_range"              value="0.1"/>
+<xacro:property name="two_d_lidar_max_range"              value="16"/>
 <!-- ............................... LOAD MACROS ................................. -->
 <xacro:include filename="$(find new_bcr_robot)/urdf/materials.xacro"/>
@@ -41,7 +41,7 @@
 	</collision>
 	<visual>
-		<origin xyz="0 0 0" rpy="0 0 0" />
+		<origin xyz="0 0 -0.08" rpy="0 0 0" />
   		<geometry>
-    		<box size="${chassis_length} ${chassis_width} ${chassis_height}"/>
+    		<mesh filename="package://new_bcr_robot/meshes/bcr_chassis.dae" scale="0.1 0.1 0.1"/>
   		</geometry>
 	</visual>
@@ -51,9 +51,9 @@
 	</inertial>
 </link>
-    <joint name="base_joint" type="fixed">
-      <parent link="base_ref"/>
-      <child link="base_link"/>
-      <origin xyz="0.0 0 0.0" rpy="0 0 0.0" />
-    </joint>
+<joint name="base_joint" type="fixed">
+	<parent link="base_ref"/>
+	<child link="base_link"/>
+	<origin xyz="0.0 0 0.0" rpy="0 0 0.0" />
+</joint>
 <!-- ................................ WHEELS ..................................... -->
 <xacro:trolley_wheel cardinality="front" dexterity="left"  origin_x="${chassis_length/2}" origin_y="${trolley_wheel_base/2}" origin_z="-${trolley_wheel_radius+chassis_height/2}"/>
@@ -88,5 +88,5 @@
       <parent link="base_link"/>
       <child link="two_d_lidar"/>
-      <origin xyz="0.3 0 0.45" rpy="0 0 ${-pi/2}" />
+      <origin xyz="0.3 0 0.2" rpy="0 0 ${-pi/2}" />
     </joint>
    <gazebo reference="two_d_lidar">

Commit message: Added Kinect Plugin

File: urdf/gazebo.xacro (robot description, xacro)
@@ -90,4 +90,44 @@
    </gazebo>
 </xacro:if>
+<!-- ........................... CAMERA PLUGIN ................................... -->
+<xacro:if value="$(arg camera_enabled)">
+	<gazebo reference="kinect_camera">
+		<sensor type="depth" name="kinect_camera">
+			<always_on>true</always_on>
+			<update_rate>30.0</update_rate>
+			<camera>
+				<horizontal_fov>${radians(camera_horizontal_fov)}</horizontal_fov>
+				<image>
+				<format>R8G8B8</format>
+				<width>640</width>
+				<height>480</height>
+				</image>
+				<clip>
+				<near>0.05</near>
+				<far>8.0</far>
+				</clip>
+			</camera>
+			<plugin name="kinect_camera_controller" filename="libgazebo_ros_openni_kinect.so">
+				<cameraName>kinect_camera</cameraName>
+				<alwaysOn>true</alwaysOn>
+				<updateRate>10</updateRate>
+				<imageTopicName>rgb/image_raw</imageTopicName>
+				<depthImageTopicName>depth/image_raw</depthImageTopicName>
+				<pointCloudTopicName>depth/points</pointCloudTopicName>
+				<cameraInfoTopicName>rgb/camera_info</cameraInfoTopicName>
+				<depthImageCameraInfoTopicName>depth/camera_info</depthImageCameraInfoTopicName>
+				<frameName>kinect_camera_optical</frameName>
+				<baseline>0.1</baseline>
+				<distortion_k1>0.0</distortion_k1>
+				<distortion_k2>0.0</distortion_k2>
+				<distortion_k3>0.0</distortion_k3>
+				<distortion_t1>0.0</distortion_t1>
+				<distortion_t2>0.0</distortion_t2>
+				<pointCloudCutoff>0.4</pointCloudCutoff>
+				<robotNamespace>/</robotNamespace>
+			</plugin>
+			</sensor>
+	</gazebo>
+</xacro:if>
 <!--................................................................................. -->
 </robot>

File: urdf/new_bcr_robot.xacro (robot description, xacro)
@@ -3,8 +3,7 @@
 <!--................................ XACRO CONSTANTS .............................. -->
 <xacro:property name="chassis_mass"                    		value="70"/>
-<xacro:property name="chassis_length"                    	value="0.95"/>
+<xacro:property name="chassis_length"                    	value="0.9"/>
 <xacro:property name="chassis_width"                    	value="0.64"/>
 <xacro:property name="chassis_height"                    	value="0.25"/>
-<xacro:property name="chassis_ground_clearance"           value="0.5"/>
 <xacro:property name="traction_wheel_mass"                value="1"/>
 <xacro:property name="traction_wheel_base"                value="0.88"/>
@@ -27,4 +26,8 @@
 <xacro:property name="two_d_lidar_min_range"              value="0.1"/>
 <xacro:property name="two_d_lidar_max_range"              value="16"/>
+<xacro:arg      name="camera_enabled"                 		default="false" />
+<xacro:property name="camera_baseline"                		value="0.06"/>
+<xacro:property name="camera_height"                  		value="0.10"/>
+<xacro:property name="camera_horizontal_fov"         	 		value="60"/>
 <!-- ............................... LOAD MACROS ................................. -->
 <xacro:include filename="$(find new_bcr_robot)/urdf/materials.xacro"/>
@@ -94,3 +97,38 @@
    </gazebo>
 </xacro:if>
+<!-- ............................. CAMERA ........................................ -->
+<xacro:if value="$(arg camera_enabled)">
+	<!-- KINECT CAMERA -->
+	<link name="kinect_camera">
+		<collision>
+			<origin xyz="0 0 0" rpy="0 0 0" />
+				<geometry>
+					<box size="0.07 0.3 0.09"/>
+				</geometry>
+		</collision>
+		<visual>
+			<origin xyz="0 0 0" rpy="0 0 0" />
+				<geometry>
+					<mesh filename="package://new_bcr_robot/meshes/kinect/d415.dae"/>
+				</geometry>
+				<material name="black"/>
+		</visual>
+		<inertial>
+				<mass value="0.01"/>
+				<xacro:box_inertia m="0.01" x="0.07" y="0.3" z = "0.09"/>
+		</inertial>
+	</link>
+	<joint name="kinect_camera_joint" type="fixed">
+			<origin rpy="0 0 0" xyz="${chassis_length/2} 0 ${chassis_height/4}"/>
+			<parent link="base_link"/>
+			<child link="kinect_camera"/>
+	</joint>
+<!-- 	<link name="kinect_camera_optical"/>
+	<joint name="kinect_camera_optical_joint" type="fixed">
+		<origin xyz="0 0 0" rpy="-${pi/2} 0 -${pi/2}"/>
+		<parent link="kinect_camera"/>
+		<child link="kinect_camera_optical"/>
+	</joint> -->
+</xacro:if>
+<!-- ......................................................................... -->
 </robot>
