Commit message: Gazebo plugin publishing joint states

File: urdf/gazebo.xacro (robot description, xacro)
@@ -8,6 +8,6 @@
 	<plugin name="diffdrive_plugin_multiwheel_middle" filename="libgazebo_ros_diff_drive.so">
 		<robotNamespace></robotNamespace>
-    <legacyMode>false</legacyMode>
-		<updateRate>100.0</updateRate>
+        <legacyMode>false</legacyMode>
+	    <updateRate>30</updateRate>
 		<leftJoint>middle_left_wheel_joint</leftJoint>
 		<rightJoint>middle_right_wheel_joint</rightJoint>
@@ -17,5 +17,5 @@
 		<wheelTorque>${traction_wheel_torque}</wheelTorque>
 		<commandTopic>/cmd_vel</commandTopic>
-		<odometryTopic>/odom</odometryTopic>
+		<odometryTopic>/diff_drive/odometry</odometryTopic>
 		<odometryFrame>odom</odometryFrame>
 		<rosDebugLevel>na</rosDebugLevel>
@@ -23,8 +23,8 @@
 		<publishOdomTF>true</publishOdomTF>
 		<publishWheelTF>false</publishWheelTF>
-		<publishWheelJointState>false</publishWheelJointState>
+		<publishWheelJointState>true</publishWheelJointState>
 		<publishOdometryMsg>true</publishOdometryMsg>
 		<odometrySource>world</odometrySource>
-    <wheelAcceleration>5.0</wheelAcceleration>
+        <wheelAcceleration>5.0</wheelAcceleration>
 	</plugin>
 </gazebo>
@@ -32,24 +32,35 @@
 <gazebo>
 	<plugin name="imu_plugin" filename="libgazebo_ros_imu.so">
-			<updateRate>50.0</updateRate>
-			<bodyName>base_link</bodyName>
-			<topicName>/imu</topicName>
-			<serviceName>/imu/calibrate</serviceName>
-			<accelOffset>0.0 0.0 0.0</accelOffset>
-			<accelDrift>0.0 0.0 0.0</accelDrift>
-			<accelDriftFrequency>0.0 0.0 0.0</accelDriftFrequency>
-			<accelGaussianNoise>0.0 0.0 0.0</accelGaussianNoise>
-			<rateOffset>0.0 0.0 0.0</rateOffset>
-			<rateDrift>0.0 0.0 0.0</rateDrift>
-			<rateDriftFrequency>0.0 0.0 0.0</rateDriftFrequency>
-			<rateGaussianNoise>0.0 0.0 0.0</rateGaussianNoise>
-			<headingOffset>0.0</headingOffset>
-			<headingDrift>0.0</headingDrift>
-			<headingDriftFrequency>0.0</headingDriftFrequency>
-			<headingGaussianNoise>0.0</headingGaussianNoise>
-			<rpyOffset>0.0 0.0 0.0</rpyOffset>
-			<xyzOffset>0.0 0.0 0.0</xyzOffset>
-			<gaussianNoise>0.0</gaussianNoise>
-			<frameName>imu_frame</frameName>
+		<updateRate>30.0</updateRate>
+		<bodyName>base_link</bodyName>
+		<topicName>/imu</topicName>
+		<serviceName>/imu/calibrate</serviceName>
+		<accelOffset>0.0 0.0 0.0</accelOffset>
+		<accelDrift>0.0 0.0 0.0</accelDrift>
+		<accelDriftFrequency>0.0 0.0 0.0</accelDriftFrequency>
+		<accelGaussianNoise>0.0 0.0 0.0</accelGaussianNoise>
+		<rateOffset>0.0 0.0 0.0</rateOffset>
+		<rateDrift>0.0 0.0 0.0</rateDrift>
+		<rateDriftFrequency>0.0 0.0 0.0</rateDriftFrequency>
+		<rateGaussianNoise>0.0 0.0 0.0</rateGaussianNoise>
+		<headingOffset>0.0</headingOffset>
+		<headingDrift>0.0</headingDrift>
+		<headingDriftFrequency>0.0</headingDriftFrequency>
+		<headingGaussianNoise>0.0</headingGaussianNoise>
+		<rpyOffset>0.0 0.0 0.0</rpyOffset>
+		<xyzOffset>0.0 0.0 0.0</xyzOffset>
+		<gaussianNoise>0.0</gaussianNoise>
+		<frameName>imu_frame</frameName>
+	</plugin>
+</gazebo>
+<!--............................... Ground truth PLUGIN .............................-->
+<gazebo>
+	<plugin name="p3d_base_controller" filename="libgazebo_ros_p3d.so">
+		<alwaysOn>true</alwaysOn>
+		<updateRate>30.0</updateRate>
+		<bodyName>base_link</bodyName>
+		<topicName>ground_truth</topicName>
+		<gaussianNoise>0.00</gaussianNoise>
+		<frameName>map</frameName>
 	</plugin>
 </gazebo>
@@ -127,5 +138,5 @@
 				<robotNamespace>/</robotNamespace>
 			</plugin>
-			</sensor>
+		</sensor>
 	</gazebo>
 </xacro:if>

File: urdf/new_bcr_robot.xacro (robot description, xacro)
@@ -35,6 +35,6 @@
 <xacro:include filename="$(find new_bcr_robot)/urdf/gazebo.xacro"/>
 <!-- ................................ BASE LINK .................................. -->
-<link name="base_ref"/>
-<link name="base_link">
+<link name="base_link"/>
+<link name="chassis_link">
 	<collision>
 		<origin xyz="0 0 0" rpy="0 0 0" />
@@ -54,7 +54,7 @@
 	</inertial>
 </link>
-<joint name="base_joint" type="fixed">
-	<parent link="base_ref"/>
-	<child link="base_link"/>
+<joint name="chassis_joint" type="fixed">
+	<parent link="base_link"/>
+	<child link="chassis_link"/>
 	<origin xyz="0.0 0 0.0" rpy="0 0 0.0" />
 </joint>
@@ -124,10 +124,10 @@
 			<child link="kinect_camera"/>
 	</joint>
-<!-- 	<link name="kinect_camera_optical"/>
+	<link name="kinect_camera_optical"/>
 	<joint name="kinect_camera_optical_joint" type="fixed">
 		<origin xyz="0 0 0" rpy="-${pi/2} 0 -${pi/2}"/>
 		<parent link="kinect_camera"/>
 		<child link="kinect_camera_optical"/>
-	</joint> -->
+	</joint>
 </xacro:if>
 <!-- ......................................................................... -->

Commit message: odom topic as argument

File: urdf/gazebo.xacro (robot description, xacro)
@@ -9,5 +9,5 @@
 		<robotNamespace></robotNamespace>
         <legacyMode>false</legacyMode>
-	    <updateRate>30</updateRate>
+	    <updateRate>100.0</updateRate>
 		<leftJoint>middle_left_wheel_joint</leftJoint>
 		<rightJoint>middle_right_wheel_joint</rightJoint>
@@ -17,5 +17,5 @@
 		<wheelTorque>${traction_wheel_torque}</wheelTorque>
 		<commandTopic>/cmd_vel</commandTopic>
-		<odometryTopic>/diff_drive/odometry</odometryTopic>
+		<odometryTopic>${wheel_odom_topic}</odometryTopic>
 		<odometryFrame>odom</odometryFrame>
 		<rosDebugLevel>na</rosDebugLevel>
@@ -32,5 +32,5 @@
 <gazebo>
 	<plugin name="imu_plugin" filename="libgazebo_ros_imu.so">
-		<updateRate>30.0</updateRate>
+		<updateRate>50.0</updateRate>
 		<bodyName>base_link</bodyName>
 		<topicName>/imu</topicName>
@@ -60,6 +60,7 @@
 		<updateRate>30.0</updateRate>
 		<bodyName>base_link</bodyName>
-		<topicName>ground_truth</topicName>
+		<topicName>ground_truth_pose</topicName>
 		<gaussianNoise>0.00</gaussianNoise>
+		<!-- pass in as argument-->
 		<frameName>map</frameName>
 	</plugin>

File: urdf/new_bcr_robot.xacro (robot description, xacro)
@@ -21,4 +21,5 @@
 <xacro:arg      name="two_d_lidar_enabled"                default="false" />
 <xacro:property name="two_d_lidar_update_rate"            value="30"/>
+<xacro:property name="wheel_odom_topic"            		  value="$(arg wheel_odom_topic)"/>
 <xacro:property name="two_d_lidar_sample_size"            value="361"/>
 <xacro:property name="two_d_lidar_min_angle"              value="0"/>

Commit message: ROS2 Branch

File: urdf/gazebo.xacro (robot description, xacro)
@@ -6,26 +6,24 @@
 <!-- .....................MULTI WHEEL DIFF DRIVE ................................... -->
 <gazebo>
-	<plugin name="diffdrive_plugin_multiwheel_middle" filename="libgazebo_ros_diff_drive.so">
-		<robotNamespace></robotNamespace>
-        <legacyMode>false</legacyMode>
-	    <updateRate>50.0</updateRate>
-		<leftJoint>middle_left_wheel_joint</leftJoint>
-		<rightJoint>middle_right_wheel_joint</rightJoint>
-		<wheelSeparation>${traction_wheel_base+traction_wheel_width-0.01}</wheelSeparation>
-		<wheelDiameter>${2*traction_wheel_radius+0.01}</wheelDiameter>
-		<robotBaseFrame>base_link</robotBaseFrame>
-		<wheelTorque>${traction_wheel_torque}</wheelTorque>
-		<commandTopic>cmd_vel</commandTopic>
-		<odometryTopic>${wheel_odom_topic}</odometryTopic>
-		<odometryFrame>odom</odometryFrame>
-		<rosDebugLevel>na</rosDebugLevel>
+	<plugin name="diff_drive" filename="libgazebo_ros_diff_drive.so">
+        <legacy_mode>false</legacy_mode>
+	    <update_rate>50.0</update_rate>
+		<left_joint>middle_left_wheel_joint</left_joint>
+		<right_joint>middle_right_wheel_joint</right_joint>
+		<wheel_separation>${traction_wheel_base+traction_wheel_width-0.01}</wheel_separation>
+		<wheel_diameter>${2*traction_wheel_radius+0.01}</wheel_diameter>
+		<robot_base_frame>base_link</robot_base_frame>
+		<max_wheel_torque>${traction_max_wheel_torque}</max_wheel_torque>
+		<command_topic>cmd_vel</command_topic>
+		<odometry_topic>${wheel_odom_topic}</odometry_topic>
+		<odometry_frame>odom</odometry_frame>
 		<xacro:unless value="$(arg publish_wheel_odom_tf)">
-			<publishOdomTF>false</publishOdomTF>
+			<publish_odom_tf>false</publish_odom_tf>
 		</xacro:unless>
-		<publishWheelTF>false</publishWheelTF>
-		<publishWheelJointState>true</publishWheelJointState>
-		<publishOdometryMsg>true</publishOdometryMsg>
-		<odometrySource>encoder</odometrySource>
-        <wheelAcceleration>5.0</wheelAcceleration>
+		<publish_wheel_tf>false</publish_wheel_tf>
+		<!-- <publish_wheel_joint_state>true</publish_wheel_joint_state> -->
+		<publish_odom>true</publish_odom>
+		<!-- <odometry_source>encoder</odometry_source> -->
+        <max_wheel_acceleration>5.0</max_wheel_acceleration>
 	</plugin>
 </gazebo>
@@ -56,14 +54,14 @@
 </gazebo> -->
 <!--............................... Ground truth PLUGIN .............................-->
-<gazebo>
+<!-- <gazebo>
 	<plugin name="p3d_base_controller" filename="libgazebo_ros_p3d.so">
-		<alwaysOn>true</alwaysOn>
-		<updateRate>30.0</updateRate>
-		<bodyName>base_link</bodyName>
-		<topicName>ground_truth_pose</topicName>
-		<gaussianNoise>0.00</gaussianNoise>
-		<frameName>$(arg ground_truth_frame)</frameName>
+		<always_on>true</always_on>
+		<update_rate>30.0</update_rate>
+		<body_name>base_link</body_name>
+		<topic_name>ground_truth_pose</topic_name>
+		<gaussian_noise>0.00</gaussian_noise>
+		<frame_name>$(arg ground_truth_frame)</frame_name>
 	</plugin>
-</gazebo>
+</gazebo> -->
 <!-- ........................... 2D LIDAR PLUGIN ................................... -->
 <xacro:if value="$(arg two_d_lidar_enabled)">

File: urdf/new_bcr_robot.xacro (robot description, xacro)
@@ -8,5 +8,5 @@
 <xacro:property name="traction_wheel_mass"                value="1"/>
 <xacro:property name="traction_wheel_base"                value="0.88"/>
-<xacro:property name="traction_wheel_torque"              value="20000"/>
+<xacro:property name="traction_max_wheel_torque"              value="20000"/>
 <xacro:property name="traction_wheel_friction"            value="5.0"/>
 <xacro:property name="trolley_wheel_mass"                 value="0.1"/>
@@ -50,5 +50,5 @@
 		<origin xyz="0 0 -0.08" rpy="0 0 0" />
   		<geometry>
-    		<mesh filename="package://new_bcr_robot/meshes/bcr_chassis.dae" scale="0.1 0.1 0.1"/>
+    		<mesh filename="file://$(find new_bcr_robot)/meshes/bcr_chassis.dae" scale="0.1 0.1 0.1"/>
   		</geometry>
 	</visual>
@@ -114,5 +114,5 @@
 			<origin xyz="0 0 0" rpy="0 0 0" />
 				<geometry>
-					<mesh filename="package://new_bcr_robot/meshes/kinect/d415.dae"/>
+					<mesh filename="file://$(find new_bcr_robot)/meshes/kinect/d415.dae"/>
 				</geometry>
 				<material name="black"/>

Commit message: Fixing Inertia Macros and wheel odom topic input

File: urdf/gazebo.xacro (robot description, xacro)
@@ -16,5 +16,5 @@
 		<max_wheel_torque>${traction_max_wheel_torque}</max_wheel_torque>
 		<command_topic>cmd_vel</command_topic>
-		<odometry_topic>${wheel_odom_topic}</odometry_topic>
+		<odometry_topic>$(arg wheel_odom_topic)</odometry_topic>
 		<odometry_frame>odom</odometry_frame>
 		<xacro:unless value="$(arg publish_wheel_odom_tf)">

File: urdf/gz.xacro (robot description, xacro)
@@ -12,5 +12,5 @@
         <odom_publish_frequency>30</odom_publish_frequency>
         <topic>/cmd_vel</topic>
-        <odom_topic>${wheel_odom_topic}</odom_topic>
+        <odom_topic>$(arg wheel_odom_topic)</odom_topic>
         <tf_topic>/tf</tf_topic>
         <frame_id>odom</frame_id>

File: urdf/macros.xacro (robot description, xacro)
@@ -11,5 +11,5 @@
     <inertia ixx="${m * (y * y + z * z) / 12}" ixy="0" ixz="0"
       iyy="${m * (x * x + z * z) / 12}" iyz="0"
-      izz="${m * (x * x + z * z) / 12}"
+      izz="${m * (y * y + x * x) / 12}"
     />
   </xacro:macro>

File: urdf/new_bcr_robot.xacro (robot description, xacro)
@@ -19,7 +19,5 @@
 <xacro:property name="traction_wheel_width"        value="0.05"/>
 <xacro:property name="traction_wheel_base"         value="0.8"/>
-<xacro:arg      name="two_d_lidar_enabled"         default="false" />
 <xacro:property name="two_d_lidar_update_rate"     value="30"/>
-<xacro:property name="wheel_odom_topic"            value="$(arg wheel_odom_topic)"/>
 <xacro:property name="two_d_lidar_sample_size"     value="361"/>
 <xacro:property name="two_d_lidar_min_angle"       value="0"/>
@@ -27,8 +25,10 @@
 <xacro:property name="two_d_lidar_min_range"       value="0.1"/>
 <xacro:property name="two_d_lidar_max_range"       value="16"/>
-<xacro:arg      name="camera_enabled"              default="false" />
 <xacro:property name="camera_baseline"             value="0.06"/>
 <xacro:property name="camera_height"               value="0.10"/>
 <xacro:property name="camera_horizontal_fov"       value="60"/>
+<xacro:arg      name="wheel_odom_topic"            default="odom" />
+<xacro:arg      name="camera_enabled"              default="false" />
+<xacro:arg      name="two_d_lidar_enabled"         default="false" />
 <xacro:arg      name="publish_wheel_odom_tf"       default="true" />
 <xacro:arg      name="conveyor_enabled"            default="false"/>
