Commit message: Styling, Cleaning and Docs

File: urdf/gazebo.xacro (robot description, xacro)
@@ -7,7 +7,7 @@
 <gazebo>
 	<plugin name="diffdrive_plugin_multiwheel_middle" filename="libgazebo_ros_diff_drive.so">
-		<robotNamespace></robotNamespace>
-        <legacyMode>false</legacyMode>
-	    <updateRate>50.0</updateRate>
+		<robotNamespace>$(arg robot_namespace)</robotNamespace>
+		<legacyMode>false</legacyMode>
+		<updateRate>50.0</updateRate>
 		<leftJoint>middle_left_wheel_joint</leftJoint>
 		<rightJoint>middle_right_wheel_joint</rightJoint>
@@ -15,7 +15,7 @@
 		<wheelDiameter>${2*traction_wheel_radius+0.01}</wheelDiameter>
 		<robotBaseFrame>base_link</robotBaseFrame>
-		<wheelTorque>${traction_wheel_torque}</wheelTorque>
+		<wheelTorque>${traction_max_wheel_torque}</wheelTorque>
 		<commandTopic>cmd_vel</commandTopic>
-		<odometryTopic>${wheel_odom_topic}</odometryTopic>
+		<odometryTopic>$(arg wheel_odom_topic)</odometryTopic>
 		<odometryFrame>odom</odometryFrame>
 		<rosDebugLevel>na</rosDebugLevel>
@@ -27,5 +27,5 @@
 		<publishOdometryMsg>true</publishOdometryMsg>
 		<odometrySource>encoder</odometrySource>
-        <wheelAcceleration>5.0</wheelAcceleration>
+		<wheelAcceleration>5.0</wheelAcceleration>
 	</plugin>
 </gazebo>
@@ -34,4 +34,5 @@
 	<plugin name="imu_plugin" filename="libgazebo_ros_imu.so">
 		<updateRate>50.0</updateRate>
+		<robotNamespace>$(arg robot_namespace)</robotNamespace>
 		<bodyName>base_link</bodyName>
 		<topicName>/imu</topicName>
@@ -58,4 +59,5 @@
 <gazebo>
 	<plugin name="p3d_base_controller" filename="libgazebo_ros_p3d.so">
+		<robotNamespace>$(arg robot_namespace)</robotNamespace>
 		<alwaysOn>true</alwaysOn>
 		<updateRate>30.0</updateRate>
@@ -68,37 +70,37 @@
 <!-- ........................... 2D LIDAR PLUGIN ................................... -->
 <xacro:if value="$(arg two_d_lidar_enabled)">
-   <gazebo reference="two_d_lidar">
-      <gravity>true</gravity>
-      <sensor type="ray" name="two_d_lidar">
-        <pose>0 0 0 0 0 0</pose>
-        <visualize>false</visualize>
-        <update_rate>${two_d_lidar_update_rate}</update_rate>
-        <ray>
-          <scan>
-            <horizontal>
-              <samples>${two_d_lidar_sample_size}</samples>
-              <resolution>1</resolution>
-              <min_angle>${radians(two_d_lidar_min_angle)}</min_angle>
-              <max_angle>${radians(two_d_lidar_max_angle)}</max_angle>
-            </horizontal>
-          </scan>
-          <range>
-            <min>${two_d_lidar_min_range}</min>
-            <max>${two_d_lidar_max_range}</max>
-            <resolution>0.01</resolution>
-          </range>
-          <noise>
-            <type>gaussian</type>
-            <mean>0.0</mean>
-            <stddev>0.001</stddev>
-          </noise>
-        </ray>
-        <plugin name="gazebo_ros_laser" filename="libgazebo_ros_laser.so">
-          <topicName>scan</topicName>
-          <frameName>two_d_lidar</frameName>
-          <robotNamespace>/</robotNamespace>
-        </plugin>
-      </sensor>
-   </gazebo>
+    <gazebo reference="two_d_lidar">
+		<gravity>true</gravity>
+		<sensor type="ray" name="two_d_lidar">
+			<pose>0 0 0 0 0 0</pose>
+			<visualize>false</visualize>
+			<update_rate>${two_d_lidar_update_rate}</update_rate>
+			<ray>
+				<scan>
+					<horizontal>
+						<samples>${two_d_lidar_sample_size}</samples>
+						<resolution>1</resolution>
+						<min_angle>${radians(two_d_lidar_min_angle)}</min_angle>
+						<max_angle>${radians(two_d_lidar_max_angle)}</max_angle>
+					</horizontal>
+				</scan>
+				<range>
+					<min>${two_d_lidar_min_range}</min>
+					<max>${two_d_lidar_max_range}</max>
+					<resolution>0.01</resolution>
+				</range>
+				<noise>
+					<type>gaussian</type>
+					<mean>0.0</mean>
+					<stddev>0.001</stddev>
+				</noise>
+			</ray>
+			<plugin name="gazebo_ros_laser" filename="libgazebo_ros_laser.so">
+				<topicName>scan</topicName>
+				<frameName>two_d_lidar</frameName>
+				<robotNamespace>$(arg robot_namespace)</robotNamespace>
+			</plugin>
+		</sensor>
+    </gazebo>
 </xacro:if>
 <!-- ........................... CAMERA PLUGIN ................................... -->
@@ -111,11 +113,11 @@
 				<horizontal_fov>${radians(camera_horizontal_fov)}</horizontal_fov>
 				<image>
-				<format>R8G8B8</format>
-				<width>640</width>
-				<height>480</height>
+					<format>R8G8B8</format>
+					<width>640</width>
+					<height>480</height>
 				</image>
 				<clip>
-				<near>0.05</near>
-				<far>8.0</far>
+					<near>0.05</near>
+					<far>8.0</far>
 				</clip>
 			</camera>
@@ -137,5 +139,5 @@
 				<distortion_t2>0.0</distortion_t2>
 				<pointCloudCutoff>0.4</pointCloudCutoff>
-				<robotNamespace>/</robotNamespace>
+				<robotNamespace>$(arg robot_namespace)</robotNamespace>
 			</plugin>
 		</sensor>

File: urdf/macros.xacro (robot description, xacro)
@@ -2,72 +2,72 @@
 <robot xmlns:xacro="http://www.ros.org/wiki/xacro" name="new_bcr_robot">
 <!--................................ INERTIA MATRICES .............................. -->
-  <xacro:macro name="cylinder_inertia" params="m r h">
-    <inertia ixx="${m * (3 * r * r + h * h) / 12}" ixy="0" ixz="0"
-      iyy="${m * (3 * r * r + h * h) / 12}" iyz="0"
-      izz="${m * r * r / 2}"
-    />
-  </xacro:macro>
-  <xacro:macro name="box_inertia" params="m x y z">
-    <inertia ixx="${m * (y * y + z * z) / 12}" ixy="0" ixz="0"
-      iyy="${m * (x * x + z * z) / 12}" iyz="0"
-      izz="${m * (x * x + z * z) / 12}"
-    />
-  </xacro:macro>
-  <xacro:macro name="sphere_inertia" params="m r">
-    <inertia ixx="${2 * m * r * r / 5}" ixy="0" ixz="0"
-      iyy="${2 * m * r * r / 5}" iyz="0"
-      izz="${2 * m * r * r / 5}"
-    />
-  </xacro:macro>
+<xacro:macro name="cylinder_inertia" params="m r h">
+	<inertia ixx="${m * (3 * r * r + h * h) / 12}" ixy="0" ixz="0"
+		iyy="${m * (3 * r * r + h * h) / 12}" iyz="0"
+		izz="${m * r * r / 2}"
+	/>
+</xacro:macro>
+<xacro:macro name="box_inertia" params="m x y z">
+	<inertia ixx="${m * (y * y + z * z) / 12}" ixy="0" ixz="0"
+		iyy="${m * (x * x + z * z) / 12}" iyz="0"
+		izz="${m * (y * y + x * x) / 12}"
+	/>
+</xacro:macro>
+<xacro:macro name="sphere_inertia" params="m r">
+	<inertia ixx="${2 * m * r * r / 5}" ixy="0" ixz="0"
+	iyy="${2 * m * r * r / 5}" iyz="0"
+	izz="${2 * m * r * r / 5}"
+	/>
+</xacro:macro>
 <!-- ............................... TROLLEY WHEEL DEFINITION .............................. -->
- <xacro:macro name="trolley_wheel" params="cardinality dexterity origin_x origin_y origin_z">
-   <link name="${cardinality}_${dexterity}_wheel">
-    <collision>
-      <origin xyz="0 0 0" rpy="0 ${pi/2} ${pi/2}" />
-      <geometry>
-       <sphere radius="${trolley_wheel_radius}"/>
-      </geometry>
-    </collision>
-    <inertial>
-      <origin xyz="0 0 0" rpy="0 0 0" />
-      <mass value="${trolley_wheel_mass}"/>
-				<xacro:sphere_inertia m="${trolley_wheel_mass}" r="${trolley_wheel_radius}"/>
-    </inertial>
-    <mu>0.0</mu>
-   </link>
-   <joint name="${cardinality}_${dexterity}_wheel_joint" type="fixed">
-      <parent link="base_link"/>
-      <child link="${cardinality}_${dexterity}_wheel"/>
-      <origin xyz="${origin_x} ${origin_y} ${origin_z}" rpy="0 0 0" />
-      <axis xyz="0 1 0" rpy="0 0 0" />
-    </joint>
-   <gazebo reference="${cardinality}_${dexterity}_wheel">
-      <material>Gazebo/Black</material>
-   </gazebo>
-  </xacro:macro>
- <xacro:macro name="traction_wheel" params="cardinality dexterity origin_x origin_y origin_z">
-   <link name="${cardinality}_${dexterity}_wheel">
-    <collision>
-      <origin xyz="0 0 0" rpy="0 ${pi/2} ${pi/2}" />
-      <geometry>
-       <cylinder length="${traction_wheel_width}" radius="${traction_wheel_radius}"/>
-      </geometry>
-    </collision>
-    <inertial>
-      <origin xyz="0 0 0" rpy="0 ${pi/2} ${pi/2}" />
-      <mass value="${traction_wheel_mass}"/>
-      <xacro:cylinder_inertia m="${traction_wheel_mass}" r="${traction_wheel_radius}" h="${traction_wheel_width}"/>
-    </inertial>
-    <mu>5.0</mu>
-   </link>
-   <joint name="${cardinality}_${dexterity}_wheel_joint" type="continuous">
-      <parent link="base_link"/>
-      <child link="${cardinality}_${dexterity}_wheel"/>
-      <origin xyz="${origin_x} ${origin_y} ${origin_z}" rpy="0 0 0" />
-      <axis xyz="0 1 0" rpy="0 0 0" />
-    </joint>
-   <gazebo reference="${cardinality}_${dexterity}_wheel">
-      <material>Gazebo/Black</material>
-   </gazebo>
-  </xacro:macro>
+<xacro:macro name="trolley_wheel" params="cardinality dexterity origin_x origin_y origin_z">
+	<link name="${cardinality}_${dexterity}_wheel">
+		<collision>
+			<origin xyz="0 0 0" rpy="0 ${pi/2} ${pi/2}" />
+			<geometry>
+				<sphere radius="${trolley_wheel_radius}"/>
+			</geometry>
+		</collision>
+		<inertial>
+			<origin xyz="0 0 0" rpy="0 0 0" />
+			<mass value="${trolley_wheel_mass}"/>
+			<xacro:sphere_inertia m="${trolley_wheel_mass}" r="${trolley_wheel_radius}"/>
+		</inertial>
+		<mu>0.0</mu>
+	</link>
+	<joint name="${cardinality}_${dexterity}_wheel_joint" type="fixed">
+		<parent link="base_link"/>
+		<child link="${cardinality}_${dexterity}_wheel"/>
+		<origin xyz="${origin_x} ${origin_y} ${origin_z}" rpy="0 0 0" />
+		<axis xyz="0 1 0" rpy="0 0 0" />
+	</joint>
+	<gazebo reference="${cardinality}_${dexterity}_wheel">
+		<material>Gazebo/Black</material>
+	</gazebo>
+</xacro:macro>
+<xacro:macro name="traction_wheel" params="cardinality dexterity origin_x origin_y origin_z">
+	<link name="${cardinality}_${dexterity}_wheel">
+		<collision>
+			<origin xyz="0 0 0" rpy="0 ${pi/2} ${pi/2}" />
+			<geometry>
+				<cylinder length="${traction_wheel_width}" radius="${traction_wheel_radius}"/>
+			</geometry>
+		</collision>
+		<inertial>
+			<origin xyz="0 0 0" rpy="0 ${pi/2} ${pi/2}" />
+			<mass value="${traction_wheel_mass}"/>
+			<xacro:cylinder_inertia m="${traction_wheel_mass}" r="${traction_wheel_radius}" h="${traction_wheel_width}"/>
+		</inertial>
+		<mu>5.0</mu>
+	</link>
+	<joint name="${cardinality}_${dexterity}_wheel_joint" type="continuous">
+		<parent link="base_link"/>
+		<child link="${cardinality}_${dexterity}_wheel"/>
+		<origin xyz="${origin_x} ${origin_y} ${origin_z}" rpy="0 0 0" />
+		<axis xyz="0 1 0" rpy="0 0 0" />
+	</joint>
+	<gazebo reference="${cardinality}_${dexterity}_wheel">
+		<material>Gazebo/Black</material>
+	</gazebo>
+</xacro:macro>
 </robot>

File: urdf/materials.xacro (robot description, xacro)
@@ -1,42 +1,42 @@
 <?xml version="1.0"?>
 <robot xmlns:xacro="http://www.ros.org/wiki/xacro" name="new_bcr_robot">
-  <material name="black">
-    <color rgba="0.0 0.0 0.0 1.0"/>
-  </material>
-  <material name="blue">
-    <color rgba="0.0 0.0 0.8 1.0"/>
-  </material>
-  <material name="green">
-    <color rgba="0.0 0.8 0.0 1.0"/>
-  </material>
-  <material name="yellow">
-    <color rgba="1.0 1.0 0.0 1.0"/>
-  </material>
-  <material name="dark_grey">
-    <color rgba="0.2 0.2 0.2 1.0"/>
-  </material>
-  <material name="orange">
-    <color rgba="${255/255} ${108/255} ${10/255} 1.0"/>
-  </material>
-  <material name="brown">
-    <color rgba="${139/255} ${69/255} ${19/255} 1.0"/>
-  </material>
-  <material name="red">
-    <color rgba="0.8 0.0 0.0 1.0"/>
-  </material>
-  <material name="turquoise">
-    <color rgba="${64/255} ${224/255} ${208/255} 1.0"/>
-  </material>
-  <material name="purple">
-    <color rgba="${128/255} ${0/255} ${128/255} 1.0"/>
-  </material>
-  <material name="white">
-    <color rgba="1.0 1.0 1.0 1.0"/>
-  </material>
-  <material name="aluminium">
-    <color rgba="0.5 0.5 0.5 1"/>
-  </material>
-  <material name="plastic">
-    <color rgba="0.1 0.1 0.1 1"/>
-  </material>
+<material name="black">
+	<color rgba="0.0 0.0 0.0 1.0"/>
+</material>
+<material name="blue">
+	<color rgba="0.0 0.0 0.8 1.0"/>
+</material>
+<material name="green">
+	<color rgba="0.0 0.8 0.0 1.0"/>
+</material>
+<material name="yellow">
+	<color rgba="1.0 1.0 0.0 1.0"/>
+</material>
+<material name="dark_grey">
+	<color rgba="0.2 0.2 0.2 1.0"/>
+</material>
+<material name="orange">
+	<color rgba="${255/255} ${108/255} ${10/255} 1.0"/>
+</material>
+<material name="brown">
+	<color rgba="${139/255} ${69/255} ${19/255} 1.0"/>
+</material>
+<material name="red">
+	<color rgba="0.8 0.0 0.0 1.0"/>
+</material>
+<material name="turquoise">
+	<color rgba="${64/255} ${224/255} ${208/255} 1.0"/>
+</material>
+<material name="purple">
+	<color rgba="${128/255} ${0/255} ${128/255} 1.0"/>
+</material>
+<material name="white">
+	<color rgba="1.0 1.0 1.0 1.0"/>
+</material>
+<material name="aluminium">
+	<color rgba="0.5 0.5 0.5 1"/>
+</material>
+<material name="plastic">
+	<color rgba="0.1 0.1 0.1 1"/>
+</material>
 </robot>

File: urdf/new_bcr_robot.xacro (robot description, xacro)
@@ -2,36 +2,37 @@
 <robot xmlns:xacro="http://www.ros.org/wiki/xacro" name="new_bcr_robot">
 <!--................................ XACRO CONSTANTS .............................. -->
-<xacro:property name="chassis_mass"                    		value="70"/>
-<xacro:property name="chassis_length"                    	value="0.9"/>
-<xacro:property name="chassis_width"                    	value="0.64"/>
-<xacro:property name="chassis_height"                    	value="0.25"/>
-<xacro:property name="traction_wheel_mass"                value="1"/>
-<xacro:property name="traction_wheel_base"                value="0.88"/>
-<xacro:property name="traction_wheel_torque"              value="20000"/>
-<xacro:property name="traction_wheel_friction"            value="5.0"/>
-<xacro:property name="trolley_wheel_mass"                 value="0.1"/>
-<xacro:property name="trolley_wheel_base"                 value="0.54"/>
-<xacro:property name="trolley_wheel_friction"             value="0.0"/>
-<xacro:property name="trolley_wheel_radius"               value="0.06"/>
+<xacro:property name="chassis_mass"                value="70"/>
+<xacro:property name="chassis_length"              value="0.9"/>
+<xacro:property name="chassis_width"               value="0.64"/>
+<xacro:property name="chassis_height"              value="0.25"/>
+<xacro:property name="traction_wheel_mass"         value="1"/>
+<xacro:property name="traction_wheel_base"         value="0.88"/>
+<xacro:property name="traction_max_wheel_torque"   value="20000"/>
+<xacro:property name="traction_wheel_friction"     value="5.0"/>
+<xacro:property name="trolley_wheel_mass"          value="0.1"/>
+<xacro:property name="trolley_wheel_base"          value="0.54"/>
+<xacro:property name="trolley_wheel_friction"      value="0.0"/>
+<xacro:property name="trolley_wheel_radius"        value="0.06"/>
 <!-- a small constant -->
-<xacro:property name="eps"                                value="0.002"/>
-<xacro:property name="traction_wheel_radius"              value="0.1"/>
-<xacro:property name="traction_wheel_width"               value="0.05"/>
-<xacro:property name="traction_wheel_base"                value="0.8"/>
-<xacro:arg      name="two_d_lidar_enabled"                default="false" />
-<xacro:property name="two_d_lidar_update_rate"            value="30"/>
-<xacro:property name="wheel_odom_topic"            		  value="$(arg wheel_odom_topic)"/>
-<xacro:property name="two_d_lidar_sample_size"            value="361"/>
-<xacro:property name="two_d_lidar_min_angle"              value="0"/>
-<xacro:property name="two_d_lidar_max_angle"              value="360"/>
-<xacro:property name="two_d_lidar_min_range"              value="0.1"/>
-<xacro:property name="two_d_lidar_max_range"              value="16"/>
-<xacro:arg      name="camera_enabled"                 		default="false" />
-<xacro:property name="camera_baseline"                		value="0.06"/>
-<xacro:property name="camera_height"                  		value="0.10"/>
-<xacro:property name="camera_horizontal_fov"         	 		value="60"/>
-<xacro:arg      name="publish_wheel_odom_tf"              default="true" />
-<xacro:arg      name="conveyor_enabled"                 	  default="false"/>
-<xacro:arg      name="ground_truth_frame"                     default="map"/>
+<xacro:property name="eps"                         value="0.002"/>
+<xacro:property name="traction_wheel_radius"       value="0.1"/>
+<xacro:property name="traction_wheel_width"        value="0.05"/>
+<xacro:property name="traction_wheel_base"         value="0.8"/>
+<xacro:property name="two_d_lidar_update_rate"     value="30"/>
+<xacro:property name="two_d_lidar_sample_size"     value="361"/>
+<xacro:property name="two_d_lidar_min_angle"       value="0"/>
+<xacro:property name="two_d_lidar_max_angle"       value="360"/>
+<xacro:property name="two_d_lidar_min_range"       value="0.1"/>
+<xacro:property name="two_d_lidar_max_range"       value="16"/>
+<xacro:property name="camera_baseline"             value="0.06"/>
+<xacro:property name="camera_height"               value="0.10"/>
+<xacro:property name="camera_horizontal_fov"       value="60"/>
+<xacro:arg      name="robot_namespace"             default="/"/>
+<xacro:arg      name="wheel_odom_topic"            default="odom"/>
+<xacro:arg      name="camera_enabled"              default="false"/>
+<xacro:arg      name="two_d_lidar_enabled"         default="false"/>
+<xacro:arg      name="publish_wheel_odom_tf"       default="true"/>
+<xacro:arg      name="conveyor_enabled"            default="false"/>
+<xacro:arg      name="ground_truth_frame"          default="map"/>
 <!-- ............................... LOAD MACROS ................................. -->
 <xacro:include filename="$(find new_bcr_robot)/urdf/materials.xacro"/>
@@ -74,30 +75,30 @@
     <link name="two_d_lidar">
         <collision>
-          <origin xyz="0 0 0" rpy="0 0 0" />
-          <geometry>
-           <cylinder length="0.06" radius="0.075"/>
-          </geometry>
+			<origin xyz="0 0 0" rpy="0 0 0" />
+			<geometry>
+				<cylinder length="0.06" radius="0.075"/>
+			</geometry>
         </collision>
         <visual>
-          <origin xyz="0 0 0" rpy="0 0 0" />
-          <geometry>
-           <cylinder length="0.06" radius="0.075"/>
-          </geometry>
-          <material name="orange"/>
+			<origin xyz="0 0 0" rpy="0 0 0" />
+			<geometry>
+				<cylinder length="0.06" radius="0.075"/>
+			</geometry>
+			<material name="orange"/>
         </visual>
         <inertial>
-          <origin xyz="0 0 0" rpy="0 0 0" />
-          <mass value="0.1"/>
-          <xacro:cylinder_inertia m="0.1" r="0.075" h="0.06"/>
+			<origin xyz="0 0 0" rpy="0 0 0" />
+			<mass value="0.1"/>
+			<xacro:cylinder_inertia m="0.1" r="0.075" h="0.06"/>
         </inertial>
-   </link>
-   <joint name="two_d_lidar_joint" type="fixed">
-      <parent link="base_link"/>
-      <child link="two_d_lidar"/>
-      <origin xyz="0.3 0 0.2" rpy="0 0 ${-pi/2}" />
+	</link>
+    <joint name="two_d_lidar_joint" type="fixed">
+		<parent link="base_link"/>
+		<child link="two_d_lidar"/>
+		<origin xyz="0.3 0 0.2" rpy="0 0 ${-pi/2}" />
     </joint>
-   <gazebo reference="two_d_lidar">
-       <material>Gazebo/Orange</material>
-   </gazebo>
+	<gazebo reference="two_d_lidar">
+		<material>Gazebo/Orange</material>
+	</gazebo>
 </xacro:if>
 <!-- ............................. CAMERA ........................................ -->
@@ -107,24 +108,24 @@
 		<collision>
 			<origin xyz="0 0 0" rpy="0 0 0" />
-				<geometry>
-					<box size="0.07 0.3 0.09"/>
-				</geometry>
+			<geometry>
+				<box size="0.07 0.3 0.09"/>
+			</geometry>
 		</collision>
 		<visual>
 			<origin xyz="0 0 0" rpy="0 0 0" />
-				<geometry>
-					<mesh filename="package://new_bcr_robot/meshes/kinect/d415.dae"/>
-				</geometry>
-				<material name="black"/>
+			<geometry>
+				<mesh filename="package://new_bcr_robot/meshes/kinect/d415.dae"/>
+			</geometry>
+			<material name="black"/>
 		</visual>
 		<inertial>
-				<mass value="0.01"/>
-				<xacro:box_inertia m="0.01" x="0.07" y="0.3" z = "0.09"/>
+			<mass value="0.01"/>
+			<xacro:box_inertia m="0.01" x="0.07" y="0.3" z = "0.09"/>
 		</inertial>
 	</link>
 	<joint name="kinect_camera_joint" type="fixed">
-			<origin rpy="0 0 0" xyz="${chassis_length/2} 0 ${chassis_height/4}"/>
-			<parent link="base_link"/>
-			<child link="kinect_camera"/>
+		<origin rpy="0 0 0" xyz="${chassis_length/2} 0 ${chassis_height/4}"/>
+		<parent link="base_link"/>
+		<child link="kinect_camera"/>
 	</joint>
 	<link name="kinect_camera_optical"/>
@@ -141,5 +142,5 @@
 			<origin xyz="0 0 0" rpy="0 0 0" />
 			<geometry>
-			<box size="1 0.6 0.015"/>
+				<box size="1 0.6 0.015"/>
 			</geometry>
 		</collision>
@@ -147,5 +148,5 @@
 			<origin xyz="0 0 0" rpy="0 0 0"/>
 			<geometry>
-			<box size="1 0.6 0.015"/>
+				<box size="1 0.6 0.015"/>
 			</geometry>
 		</visual>
