Commit message: Modified chassis desgin, Updated URDF, all the sensors working, namespace done

File: urdf/gazebo.xacro (robot description, xacro)
@@ -7,4 +7,9 @@
 <gazebo>
 	<plugin name="diff_drive" filename="libgazebo_ros_diff_drive.so">
+		 <ros>
+		  <namespace>$(arg robot_namespace)</namespace>
+		  <remapping>cmd_vel:=cmd_vel</remapping>
+		  <remapping>odom:=odom</remapping>
+		</ros>
 		<legacy_mode>false</legacy_mode>
 		<update_rate>50.0</update_rate>
@@ -55,8 +60,12 @@
 <gazebo>
 	<plugin name="p3d_base_controller" filename="libgazebo_ros_p3d.so">
+		<ros>
+			<!-- Add namespace and remap the default topic -->
+			<namespace>$(arg robot_namespace)</namespace>
+			<remapping>odom:=p3d_ground_truth</remapping>
+		</ros>
 		<always_on>true</always_on>
 		<update_rate>30.0</update_rate>
 		<body_name>base_link</body_name>
-		<topic_name>ground_truth_pose</topic_name>
 		<gaussian_noise>0.00</gaussian_noise>
 		<frame_name>$(arg ground_truth_frame)</frame_name>
@@ -88,11 +97,13 @@
 					<type>gaussian</type>
 					<mean>0.0</mean>
-					<stddev>0.001</stddev>
+					<stddev>0.0</stddev>
 				</noise>
 			</ray>
-			<plugin name="gazebo_ros_laser" filename="libgazebo_ros_laser.so">
-				<topicName>scan</topicName>
+			<plugin name="gazebo_ros_laser" filename="libgazebo_ros_ray_sensor.so">
+				<ros>
+					<remapping>~/out:=/$(arg robot_namespace)/scan</remapping>
+				</ros>
+				<output_type>sensor_msgs/LaserScan</output_type>
 				<frameName>two_d_lidar</frameName>
-				<robotNamespace>$(arg robot_namespace)</robotNamespace>
 			</plugin>
 		</sensor>
@@ -101,10 +112,11 @@
 <!-- ........................... CAMERA PLUGIN ................................... -->
 <xacro:if value="$(arg camera_enabled)">
-	<gazebo reference="kinect_camera">
-		<sensor type="depth" name="kinect_camera">
-			<always_on>true</always_on>
-			<update_rate>30.0</update_rate>
+	 <gazebo reference="kinect_camera">
+		<sensor name="kinect_camera" type="depth">
+			<pose> 0 0 0 0 0 0 </pose>
+			<visualize>true</visualize>
+			<update_rate>30</update_rate>
 			<camera>
-				<horizontal_fov>${radians(camera_horizontal_fov)}</horizontal_fov>
+				<horizontal_fov>1.089</horizontal_fov>
 				<image>
 					<format>R8G8B8</format>
@@ -117,22 +129,11 @@
 				</clip>
 			</camera>
-			<plugin name="kinect_camera_controller" filename="libgazebo_ros_openni_kinect.so">
-				<cameraName>kinect_camera</cameraName>
-				<alwaysOn>true</alwaysOn>
-				<updateRate>10</updateRate>
-				<imageTopicName>rgb/image_raw</imageTopicName>
-				<depthImageTopicName>depth/image_raw</depthImageTopicName>
-				<pointCloudTopicName>depth/points</pointCloudTopicName>
-				<cameraInfoTopicName>rgb/camera_info</cameraInfoTopicName>
-				<depthImageCameraInfoTopicName>depth/camera_info</depthImageCameraInfoTopicName>
-				<frameName>kinect_camera_optical</frameName>
-				<baseline>0.1</baseline>
-				<distortion_k1>0.0</distortion_k1>
-				<distortion_k2>0.0</distortion_k2>
-				<distortion_k3>0.0</distortion_k3>
-				<distortion_t1>0.0</distortion_t1>
-				<distortion_t2>0.0</distortion_t2>
-				<pointCloudCutoff>0.4</pointCloudCutoff>
-				<robotNamespace>$(arg robot_namespace)</robotNamespace>
+			<plugin name="camera_controller" filename="libgazebo_ros_camera.so">
+				<ros>
+					<namespace>$(arg robot_namespace)</namespace>
+				</ros>
+				<frame_name>kinect_camera_optical</frame_name>
+				<min_depth>0.1</min_depth>
+				<max_depth>100</max_depth>
 			</plugin>
 		</sensor>

File: urdf/gz.xacro (robot description, xacro)
@@ -1,8 +1,10 @@
 <?xml version="1.0"?>
 <robot xmlns:xacro="http://www.ros.org/wiki/xacro" name="new_bcr_robot">
+<!-- ........................... SENSOR PLUGIN ................................... -->
 <gazebo>
     <plugin filename="ignition-gazebo-sensors-system" name="ignition::gazebo::systems::Sensors">
         <render_engine>ogre2</render_engine>
     </plugin>
+<!-- ........................... DIFFERENTIAL DRIVE PLUGIN ................................... -->
     <plugin filename="ignition-gazebo-diff-drive-system" name="ignition::gazebo::systems::DiffDrive">
         <left_joint>middle_left_wheel_joint</left_joint>
@@ -18,4 +20,5 @@
     </plugin>
 </gazebo>
+<!-- ........................... 2D LIDAR config ................................... -->
 <xacro:if value="$(arg two_d_lidar_enabled)">
     <gazebo reference="two_d_lidar">
@@ -49,4 +52,5 @@
     </gazebo>
 </xacro:if>
+<!-- ........................... CAMERA config ................................... -->
 <xacro:if value="$(arg camera_enabled)">
     <gazebo reference="kinect_camera">

File: urdf/new_bcr_robot.xacro (robot description, xacro)
@@ -5,5 +5,5 @@
 <xacro:property name="chassis_length"              value="0.9"/>
 <xacro:property name="chassis_width"               value="0.64"/>
-<xacro:property name="chassis_height"              value="0.25"/>
+<xacro:property name="chassis_height"              value="0.19"/>
 <xacro:property name="traction_wheel_mass"         value="1"/>
 <xacro:property name="traction_wheel_base"         value="0.88"/>
@@ -28,5 +28,5 @@
 <xacro:property name="camera_height"               value="0.10"/>
 <xacro:property name="camera_horizontal_fov"       value="60"/>
-<xacro:arg      name="robot_namespace"             default="/"/>
+<xacro:arg      name="robot_namespace"             default="new_bcr_robot"/>
 <xacro:arg      name="wheel_odom_topic"            default="odom" />
 <xacro:arg      name="camera_enabled"              default="false" />
@@ -50,5 +50,5 @@
 <link name="chassis_link">
 	<collision>
-		<origin xyz="0 0 0" rpy="0 0 0" />
+		<origin xyz="0 0 -0.05" rpy="0 0 0" />
   		<geometry>
 			<box size="${chassis_length} ${chassis_width} ${chassis_height}"/>
@@ -56,7 +56,7 @@
 	</collision>
 	<visual>
-		<origin xyz="0 0 -0.08" rpy="0 0 0" />
+		<origin xyz="0 0 -0.15" rpy="0 0 0" />
   		<geometry>
-    		<mesh filename="file://$(find new_bcr_robot)/meshes/bcr_chassis.dae" scale="0.1 0.1 0.1"/>
+    		<mesh filename="file://$(find new_bcr_robot)/meshes/bcr_bot_mesh.dae" scale="1 1 1"/>
   		</geometry>
 	</visual>
@@ -69,5 +69,5 @@
 	<parent link="base_link"/>
 	<child link="chassis_link"/>
-	<origin xyz="0.0 0 0.0" rpy="0 0 0.0" />
+	<origin xyz="0.0 0 0" rpy="0 0 0.0" />
 </joint>
 <!-- ................................ WHEELS ..................................... -->
@@ -92,5 +92,5 @@
            <cylinder length="0.06" radius="0.075"/>
           </geometry>
-          <material name="orange"/>
+          <material name="aluminium"/>
         </visual>
         <inertial>
@@ -103,8 +103,8 @@
       <parent link="base_link"/>
       <child link="two_d_lidar"/>
-      <origin xyz="0.3 0 0.2" rpy="0 0 ${-pi/2}" />
+      <origin xyz="0.3 0 0.08" rpy="0 0 0" />
     </joint>
    <gazebo reference="two_d_lidar">
-       <material>Gazebo/Orange</material>
+       <material>Gazebo/White</material>
    </gazebo>
 </xacro:if>
@@ -132,5 +132,5 @@
 	</link>
 	<joint name="kinect_camera_joint" type="fixed">
-			<origin rpy="0 0 0" xyz="${chassis_length/2} 0 ${chassis_height/4}"/>
+			<origin rpy="0 0 0" xyz="${chassis_length/2} 0 ${chassis_height/7}"/>
 			<parent link="base_link"/>
 			<child link="kinect_camera"/>
@@ -138,9 +138,27 @@
 	<link name="kinect_camera_optical"/>
 	<joint name="kinect_camera_optical_joint" type="fixed">
-		<origin xyz="0 0 0" rpy="-${pi/2} 0 -${pi/2}"/>
+		<origin xyz="0 0 0" rpy="${-pi/2} 0 ${-pi/2}"/>
 		<parent link="kinect_camera"/>
 		<child link="kinect_camera_optical"/>
 	</joint>
 </xacro:if>
+<!-- ............................. ROOF ........................................ -->
+<link name="roof_link">
+		<collision>
+			<origin xyz="0 0 0" rpy="0 0 0" />
+			<geometry>
+			<box size="${chassis_length} ${chassis_width} 0.015"/>
+			</geometry>
+		</collision>
+		<inertial>
+			<mass value="1"/>
+			<xacro:box_inertia m="1" x="1" y="0.6" z = "0.015"/>
+		</inertial>
+	</link>
+	<joint name="roof joint" type="fixed">
+		<parent link="chassis_link"/>
+		<child link="roof_link"/>
+		<origin xyz="0 0 0.16" rpy="0 0 0" />
+	</joint>
 <!-- ............................. CONVEYOR ........................................ -->
 <xacro:if value="$(arg conveyor_enabled)">

Commit message: New Chassis, Updated URDF, new small_warehouse World, Updated readme

File: urdf/gazebo.xacro (robot description, xacro)
@@ -20,7 +20,5 @@
 		<odometryFrame>odom</odometryFrame>
 		<rosDebugLevel>na</rosDebugLevel>
-		<xacro:unless value="$(arg publish_wheel_odom_tf)">
-			<publishOdomTF>false</publishOdomTF>
-		</xacro:unless>
+		<publishOdomTF>$(arg publish_wheel_odom_tf)</publishOdomTF>
 		<publishWheelTF>false</publishWheelTF>
 		<publishWheelJointState>true</publishWheelJointState>

File: urdf/new_bcr_robot.xacro (robot description, xacro)
@@ -5,5 +5,5 @@
 <xacro:property name="chassis_length"              value="0.9"/>
 <xacro:property name="chassis_width"               value="0.64"/>
-<xacro:property name="chassis_height"              value="0.25"/>
+<xacro:property name="chassis_height"              value="0.19"/>
 <xacro:property name="traction_wheel_mass"         value="1"/>
 <xacro:property name="traction_wheel_base"         value="0.88"/>
@@ -43,5 +43,5 @@
 <link name="chassis_link">
 	<collision>
-		<origin xyz="0 0 0" rpy="0 0 0" />
+		<origin xyz="0 0 -0.05" rpy="0 0 0" />
   		<geometry>
 			<box size="${chassis_length} ${chassis_width} ${chassis_height}"/>
@@ -49,7 +49,7 @@
 	</collision>
 	<visual>
-		<origin xyz="0 0 -0.08" rpy="0 0 0" />
+		<origin xyz="0 0 -0.2" rpy="0 0 0" />
   		<geometry>
-    		<mesh filename="package://new_bcr_robot/meshes/bcr_chassis.dae" scale="0.1 0.1 0.1"/>
+    		<mesh filename="file://$(find new_bcr_robot)/meshes/bcr_bot_mesh.dae" scale="1 1 1"/>
   		</geometry>
 	</visual>
@@ -62,5 +62,5 @@
 	<parent link="base_link"/>
 	<child link="chassis_link"/>
-	<origin xyz="0.0 0 0.0" rpy="0 0 0.0" />
+	<origin xyz="0.0 0 0" rpy="0 0 0.0" />
 </joint>
 <!-- ................................ WHEELS ..................................... -->
@@ -75,30 +75,30 @@
     <link name="two_d_lidar">
         <collision>
-			<origin xyz="0 0 0" rpy="0 0 0" />
-			<geometry>
-				<cylinder length="0.06" radius="0.075"/>
-			</geometry>
+          <origin xyz="0 0 0" rpy="0 0 0" />
+          <geometry>
+           <cylinder length="0.06" radius="0.075"/>
+          </geometry>
         </collision>
         <visual>
-			<origin xyz="0 0 0" rpy="0 0 0" />
-			<geometry>
-				<cylinder length="0.06" radius="0.075"/>
-			</geometry>
-			<material name="orange"/>
+          <origin xyz="0 0 0" rpy="0 0 0" />
+          <geometry>
+           <cylinder length="0.06" radius="0.075"/>
+          </geometry>
+          <material name="aluminium"/>
         </visual>
         <inertial>
-			<origin xyz="0 0 0" rpy="0 0 0" />
-			<mass value="0.1"/>
-			<xacro:cylinder_inertia m="0.1" r="0.075" h="0.06"/>
+          <origin xyz="0 0 0" rpy="0 0 0" />
+          <mass value="0.1"/>
+          <xacro:cylinder_inertia m="0.1" r="0.075" h="0.06"/>
         </inertial>
-	</link>
-    <joint name="two_d_lidar_joint" type="fixed">
-		<parent link="base_link"/>
-		<child link="two_d_lidar"/>
-		<origin xyz="0.3 0 0.2" rpy="0 0 ${-pi/2}" />
+   </link>
+   <joint name="two_d_lidar_joint" type="fixed">
+      <parent link="base_link"/>
+      <child link="two_d_lidar"/>
+      <origin xyz="0.3 0 0.08" rpy="0 0 0" />
     </joint>
-	<gazebo reference="two_d_lidar">
-		<material>Gazebo/Orange</material>
-	</gazebo>
+   <gazebo reference="two_d_lidar">
+       <material>Gazebo/White</material>
+   </gazebo>
 </xacro:if>
 <!-- ............................. CAMERA ........................................ -->
@@ -108,32 +108,50 @@
 		<collision>
 			<origin xyz="0 0 0" rpy="0 0 0" />
-			<geometry>
-				<box size="0.07 0.3 0.09"/>
-			</geometry>
+				<geometry>
+					<box size="0.07 0.3 0.09"/>
+				</geometry>
 		</collision>
 		<visual>
 			<origin xyz="0 0 0" rpy="0 0 0" />
-			<geometry>
-				<mesh filename="package://new_bcr_robot/meshes/kinect/d415.dae"/>
-			</geometry>
-			<material name="black"/>
+				<geometry>
+					<mesh filename="file://$(find new_bcr_robot)/meshes/kinect/d415.dae"/>
+				</geometry>
+				<material name="black"/>
 		</visual>
 		<inertial>
-			<mass value="0.01"/>
-			<xacro:box_inertia m="0.01" x="0.07" y="0.3" z = "0.09"/>
+				<mass value="0.01"/>
+				<xacro:box_inertia m="0.01" x="0.07" y="0.3" z = "0.09"/>
 		</inertial>
 	</link>
 	<joint name="kinect_camera_joint" type="fixed">
-		<origin rpy="0 0 0" xyz="${chassis_length/2} 0 ${chassis_height/4}"/>
-		<parent link="base_link"/>
-		<child link="kinect_camera"/>
+			<origin rpy="0 0 0" xyz="${chassis_length/2} 0 ${chassis_height/7}"/>
+			<parent link="base_link"/>
+			<child link="kinect_camera"/>
 	</joint>
 	<link name="kinect_camera_optical"/>
 	<joint name="kinect_camera_optical_joint" type="fixed">
-		<origin xyz="0 0 0" rpy="-${pi/2} 0 -${pi/2}"/>
+		<origin xyz="0 0 0" rpy="${-pi/2} 0 ${-pi/2}"/>
 		<parent link="kinect_camera"/>
 		<child link="kinect_camera_optical"/>
 	</joint>
 </xacro:if>
+<!-- ............................. ROOF ........................................ -->
+<link name="roof_link">
+		<collision>
+			<origin xyz="0 0 0" rpy="0 0 0" />
+			<geometry>
+			<box size="${chassis_length} ${chassis_width} 0.015"/>
+			</geometry>
+		</collision>
+		<inertial>
+			<mass value="1"/>
+			<xacro:box_inertia m="1" x="1" y="0.6" z = "0.015"/>
+		</inertial>
+	</link>
+	<joint name="roof joint" type="fixed">
+		<parent link="chassis_link"/>
+		<child link="roof_link"/>
+		<origin xyz="0 0 0.16" rpy="0 0 0" />
+	</joint>
 <!-- ............................. CONVEYOR ........................................ -->
 <xacro:if value="$(arg conveyor_enabled)">
@@ -142,5 +160,5 @@
 			<origin xyz="0 0 0" rpy="0 0 0" />
 			<geometry>
-				<box size="1 0.6 0.015"/>
+			<box size="1 0.6 0.015"/>
 			</geometry>
 		</collision>
@@ -148,5 +166,5 @@
 			<origin xyz="0 0 0" rpy="0 0 0"/>
 			<geometry>
-				<box size="1 0.6 0.015"/>
+			<box size="1 0.6 0.015"/>
 			</geometry>
 		</visual>
@@ -159,5 +177,5 @@
 		<parent link="base_link"/>
 		<child link="conveyor_belt"/>
-		<origin xyz="0 0 0.21" rpy="0 0 0" />
+		<origin xyz="0 0 0.25" rpy="0 0 0" />
 	</joint>
 </xacro:if>

Commit message: Hooks, Cleanup and Depth Camera Transform

File: urdf/gazebo.xacro (robot description, xacro)
@@ -7,8 +7,8 @@
 <gazebo>
 	<plugin name="diff_drive" filename="libgazebo_ros_diff_drive.so">
-		 <ros>
-		  <namespace>$(arg robot_namespace)</namespace>
-		  <remapping>cmd_vel:=cmd_vel</remapping>
-		  <remapping>odom:=odom</remapping>
+		<ros>
+			<namespace>$(arg robot_namespace)</namespace>
+			<remapping>cmd_vel:=cmd_vel</remapping>
+			<remapping>odom:=odom</remapping>
 		</ros>
 		<legacy_mode>false</legacy_mode>
@@ -26,5 +26,4 @@
 		<publish_wheel_tf>false</publish_wheel_tf>
 		<publish_odom>true</publish_odom>
-		<!-- <odometry_source>encoder</odometry_source> -->
 		<max_wheel_acceleration>5.0</max_wheel_acceleration>
 	</plugin>

File: urdf/macros.xacro (robot description, xacro)
@@ -2,72 +2,72 @@
 <robot xmlns:xacro="http://www.ros.org/wiki/xacro" name="new_bcr_robot">
 <!--................................ INERTIA MATRICES .............................. -->
-  <xacro:macro name="cylinder_inertia" params="m r h">
-    <inertia ixx="${m * (3 * r * r + h * h) / 12}" ixy="0" ixz="0"
-      iyy="${m * (3 * r * r + h * h) / 12}" iyz="0"
-      izz="${m * r * r / 2}"
-    />
-  </xacro:macro>
-  <xacro:macro name="box_inertia" params="m x y z">
-    <inertia ixx="${m * (y * y + z * z) / 12}" ixy="0" ixz="0"
-      iyy="${m * (x * x + z * z) / 12}" iyz="0"
-      izz="${m * (y * y + x * x) / 12}"
-    />
-  </xacro:macro>
-  <xacro:macro name="sphere_inertia" params="m r">
-    <inertia ixx="${2 * m * r * r / 5}" ixy="0" ixz="0"
-      iyy="${2 * m * r * r / 5}" iyz="0"
-      izz="${2 * m * r * r / 5}"
-    />
-  </xacro:macro>
+<xacro:macro name="cylinder_inertia" params="m r h">
+	<inertia ixx="${m * (3 * r * r + h * h) / 12}" ixy="0" ixz="0"
+		iyy="${m * (3 * r * r + h * h) / 12}" iyz="0"
+		izz="${m * r * r / 2}"
+	/>
+</xacro:macro>
+<xacro:macro name="box_inertia" params="m x y z">
+	<inertia ixx="${m * (y * y + z * z) / 12}" ixy="0" ixz="0"
+		iyy="${m * (x * x + z * z) / 12}" iyz="0"
+		izz="${m * (y * y + x * x) / 12}"
+	/>
+</xacro:macro>
+<xacro:macro name="sphere_inertia" params="m r">
+	<inertia ixx="${2 * m * r * r / 5}" ixy="0" ixz="0"
+		iyy="${2 * m * r * r / 5}" iyz="0"
+		izz="${2 * m * r * r / 5}"
+	/>
+</xacro:macro>
 <!-- ............................... TROLLEY WHEEL DEFINITION .............................. -->
- <xacro:macro name="trolley_wheel" params="cardinality dexterity origin_x origin_y origin_z">
-   <link name="${cardinality}_${dexterity}_wheel">
-    <collision>
-      <origin xyz="0 0 0" rpy="0 ${pi/2} ${pi/2}" />
-      <geometry>
-       <sphere radius="${trolley_wheel_radius}"/>
-      </geometry>
-    </collision>
-    <inertial>
-      <origin xyz="0 0 0" rpy="0 0 0" />
-      <mass value="${trolley_wheel_mass}"/>
-				<xacro:sphere_inertia m="${trolley_wheel_mass}" r="${trolley_wheel_radius}"/>
-    </inertial>
-    <mu>0.0</mu>
-   </link>
-   <joint name="${cardinality}_${dexterity}_wheel_joint" type="fixed">
-      <parent link="base_link"/>
-      <child link="${cardinality}_${dexterity}_wheel"/>
-      <origin xyz="${origin_x} ${origin_y} ${origin_z}" rpy="0 0 0" />
-      <axis xyz="0 1 0" rpy="0 0 0" />
-    </joint>
-   <gazebo reference="${cardinality}_${dexterity}_wheel">
-      <material>Gazebo/Black</material>
-   </gazebo>
-  </xacro:macro>
- <xacro:macro name="traction_wheel" params="cardinality dexterity origin_x origin_y origin_z">
-   <link name="${cardinality}_${dexterity}_wheel">
-    <collision>
-      <origin xyz="0 0 0" rpy="0 ${pi/2} ${pi/2}" />
-      <geometry>
-       <cylinder length="${traction_wheel_width}" radius="${traction_wheel_radius}"/>
-      </geometry>
-    </collision>
-    <inertial>
-      <origin xyz="0 0 0" rpy="0 ${pi/2} ${pi/2}" />
-      <mass value="${traction_wheel_mass}"/>
-      <xacro:cylinder_inertia m="${traction_wheel_mass}" r="${traction_wheel_radius}" h="${traction_wheel_width}"/>
-    </inertial>
-    <mu>5.0</mu>
-   </link>
-   <joint name="${cardinality}_${dexterity}_wheel_joint" type="continuous">
-      <parent link="base_link"/>
-      <child link="${cardinality}_${dexterity}_wheel"/>
-      <origin xyz="${origin_x} ${origin_y} ${origin_z}" rpy="0 0 0" />
-      <axis xyz="0 1 0" rpy="0 0 0" />
-    </joint>
-   <gazebo reference="${cardinality}_${dexterity}_wheel">
-      <material>Gazebo/Black</material>
-   </gazebo>
-  </xacro:macro>
+<xacro:macro name="trolley_wheel" params="cardinality dexterity origin_x origin_y origin_z">
+	<link name="${cardinality}_${dexterity}_wheel">
+		<collision>
+			<origin xyz="0 0 0" rpy="0 ${pi/2} ${pi/2}" />
+			<geometry>
+				<sphere radius="${trolley_wheel_radius}"/>
+			</geometry>
+		</collision>
+		<inertial>
+			<origin xyz="0 0 0" rpy="0 0 0" />
+			<mass value="${trolley_wheel_mass}"/>
+			<xacro:sphere_inertia m="${trolley_wheel_mass}" r="${trolley_wheel_radius}"/>
+		</inertial>
+		<mu>0.0</mu>
+	</link>
+	<joint name="${cardinality}_${dexterity}_wheel_joint" type="fixed">
+		<parent link="base_link"/>
+		<child link="${cardinality}_${dexterity}_wheel"/>
+		<origin xyz="${origin_x} ${origin_y} ${origin_z}" rpy="0 0 0" />
+		<axis xyz="0 1 0" rpy="0 0 0" />
+	</joint>
+	<gazebo reference="${cardinality}_${dexterity}_wheel">
+		<material>Gazebo/Black</material>
+	</gazebo>
+</xacro:macro>
+<xacro:macro name="traction_wheel" params="cardinality dexterity origin_x origin_y origin_z">
+	<link name="${cardinality}_${dexterity}_wheel">
+		<collision>
+			<origin xyz="0 0 0" rpy="0 ${pi/2} ${pi/2}" />
+			<geometry>
+				<cylinder length="${traction_wheel_width}" radius="${traction_wheel_radius}"/>
+			</geometry>
+		</collision>
+		<inertial>
+			<origin xyz="0 0 0" rpy="0 ${pi/2} ${pi/2}" />
+			<mass value="${traction_wheel_mass}"/>
+			<xacro:cylinder_inertia m="${traction_wheel_mass}" r="${traction_wheel_radius}" h="${traction_wheel_width}"/>
+		</inertial>
+		<mu>5.0</mu>
+	</link>
+	<joint name="${cardinality}_${dexterity}_wheel_joint" type="continuous">
+		<parent link="base_link"/>
+		<child link="${cardinality}_${dexterity}_wheel"/>
+		<origin xyz="${origin_x} ${origin_y} ${origin_z}" rpy="0 0 0" />
+		<axis xyz="0 1 0" rpy="0 0 0" />
+	</joint>
+	<gazebo reference="${cardinality}_${dexterity}_wheel">
+		<material>Gazebo/Black</material>
+	</gazebo>
+</xacro:macro>
 </robot>

File: urdf/materials.xacro (robot description, xacro)
@@ -1,42 +1,42 @@
 <?xml version="1.0"?>
 <robot xmlns:xacro="http://www.ros.org/wiki/xacro" name="new_bcr_robot">
-  <material name="black">
-    <color rgba="0.0 0.0 0.0 1.0"/>
-  </material>
-  <material name="blue">
-    <color rgba="0.0 0.0 0.8 1.0"/>
-  </material>
-  <material name="green">
-    <color rgba="0.0 0.8 0.0 1.0"/>
-  </material>
-  <material name="yellow">
-    <color rgba="1.0 1.0 0.0 1.0"/>
-  </material>
-  <material name="dark_grey">
-    <color rgba="0.2 0.2 0.2 1.0"/>
-  </material>
-  <material name="orange">
-    <color rgba="${255/255} ${108/255} ${10/255} 1.0"/>
-  </material>
-  <material name="brown">
-    <color rgba="${139/255} ${69/255} ${19/255} 1.0"/>
-  </material>
-  <material name="red">
-    <color rgba="0.8 0.0 0.0 1.0"/>
-  </material>
-  <material name="turquoise">
-    <color rgba="${64/255} ${224/255} ${208/255} 1.0"/>
-  </material>
-  <material name="purple">
-    <color rgba="${128/255} ${0/255} ${128/255} 1.0"/>
-  </material>
-  <material name="white">
-    <color rgba="1.0 1.0 1.0 1.0"/>
-  </material>
-  <material name="aluminium">
-    <color rgba="0.5 0.5 0.5 1"/>
-  </material>
-  <material name="plastic">
-    <color rgba="0.1 0.1 0.1 1"/>
-  </material>
+	<material name="black">
+		<color rgba="0.0 0.0 0.0 1.0"/>
+	</material>
+	<material name="blue">
+		<color rgba="0.0 0.0 0.8 1.0"/>
+	</material>
+	<material name="green">
+		<color rgba="0.0 0.8 0.0 1.0"/>
+	</material>
+	<material name="yellow">
+		<color rgba="1.0 1.0 0.0 1.0"/>
+	</material>
+	<material name="dark_grey">
+		<color rgba="0.2 0.2 0.2 1.0"/>
+	</material>
+	<material name="orange">
+		<color rgba="${255/255} ${108/255} ${10/255} 1.0"/>
+	</material>
+	<material name="brown">
+		<color rgba="${139/255} ${69/255} ${19/255} 1.0"/>
+	</material>
+	<material name="red">
+		<color rgba="0.8 0.0 0.0 1.0"/>
+	</material>
+	<material name="turquoise">
+		<color rgba="${64/255} ${224/255} ${208/255} 1.0"/>
+	</material>
+	<material name="purple">
+		<color rgba="${128/255} ${0/255} ${128/255} 1.0"/>
+	</material>
+	<material name="white">
+		<color rgba="1.0 1.0 1.0 1.0"/>
+	</material>
+	<material name="aluminium">
+		<color rgba="0.5 0.5 0.5 1"/>
+	</material>
+	<material name="plastic">
+		<color rgba="0.1 0.1 0.1 1"/>
+	</material>
 </robot>
