Commit message: Updated chassis with logo, Imu always on, camera and Lidar as launch param

File: urdf/gazebo.xacro (robot description, xacro)
@@ -24,5 +24,5 @@
 		<odometry_frame>odom</odometry_frame>
 		<publish_odom_tf>$(arg publish_wheel_odom_tf)</publish_odom_tf>
-		<publish_wheel_tf>false</publish_wheel_tf>
+		<publish_wheel_tf>true</publish_wheel_tf>
 		<publish_odom>true</publish_odom>
 		<max_wheel_acceleration>5.0</max_wheel_acceleration>
@@ -30,30 +30,16 @@
 </gazebo>
 <!--............................... IMU PLUGIN ..................................... -->
-<!--
-<gazebo>
-	<plugin name="imu_plugin" filename="libgazebo_ros_imu.so">
-		<updateRate>50.0</updateRate>
-		<bodyName>base_link</bodyName>
-		<topicName>/imu</topicName>
-		<serviceName>/imu/calibrate</serviceName>
-		<accelOffset>0.0 0.0 0.0</accelOffset>
-		<accelDrift>0.0 0.0 0.0</accelDrift>
-		<accelDriftFrequency>0.0 0.0 0.0</accelDriftFrequency>
-		<accelGaussianNoise>0.0 0.0 0.0</accelGaussianNoise>
-		<rateOffset>0.0 0.0 0.0</rateOffset>
-		<rateDrift>0.0 0.0 0.0</rateDrift>
-		<rateDriftFrequency>0.0 0.0 0.0</rateDriftFrequency>
-		<rateGaussianNoise>0.0 0.0 0.0</rateGaussianNoise>
-		<headingOffset>0.0</headingOffset>
-		<headingDrift>0.0</headingDrift>
-		<headingDriftFrequency>0.0</headingDriftFrequency>
-		<headingGaussianNoise>0.0</headingGaussianNoise>
-		<rpyOffset>0.0 0.0 0.0</rpyOffset>
-		<xyzOffset>0.0 0.0 0.0</xyzOffset>
-		<gaussianNoise>0.0</gaussianNoise>
-		<frameName>imu_frame</frameName>
-	</plugin>
+<gazebo reference="imu_frame">
+		<sensor name="imu" type="imu">
+			<always_on>true</always_on>
+			<update_rate>5</update_rate>
+			<plugin name="imu_plugin" filename="libgazebo_ros_imu_sensor.so">
+				<ros>
+					<namespace>$(arg robot_namespace)</namespace>
+					<remapping>~/out:=imu</remapping>
+				</ros>
+			</plugin>
+		</sensor>
 </gazebo>
--->
 <!--............................... Ground truth PLUGIN .............................-->
 <gazebo>

File: urdf/gz.xacro (robot description, xacro)
@@ -5,4 +5,7 @@
     <plugin filename="ignition-gazebo-sensors-system" name="ignition::gazebo::systems::Sensors">
         <render_engine>ogre2</render_engine>
+    </plugin>
+    <plugin filename="ignition-gazebo-imu-system"
+        name="ignition::gazebo::systems::Imu">
     </plugin>
 <!-- ........................... DIFFERENTIAL DRIVE PLUGIN ................................... -->
@@ -75,3 +78,13 @@
     </gazebo>
 </xacro:if>
+<!-- ........................... IMU config ................................... -->
+<gazebo reference="imu_frame">
+    <sensor name="imu_sensor" type="imu">
+        <always_on>1</always_on>
+        <update_rate>1</update_rate>
+        <ignition_frame_id>imu_frame</ignition_frame_id>
+        <visualize>true</visualize>
+        <topic>imu</topic>
+    </sensor>
+</gazebo>
 </robot>

File: urdf/new_bcr_robot.xacro (robot description, xacro)
@@ -56,5 +56,5 @@
 	</collision>
 	<visual>
-		<origin xyz="0 0 -0.15" rpy="0 0 0" />
+		<origin xyz="0 0 -0.205" rpy="0 0 0" />
   		<geometry>
     		<mesh filename="file://$(find new_bcr_robot)/meshes/bcr_bot_mesh.dae" scale="1 1 1"/>
@@ -109,4 +109,11 @@
    </gazebo>
 </xacro:if>
+<!-- ............................. IMU ........................................ -->
+<link name="imu_frame"/>
+<joint name="imu_joint" type="fixed">
+    <parent link="base_link"/>
+    <child link="imu_frame"/>
+    <origin xyz="0.0 0.0 0.08" rpy="0.0 0.0 0.0"/>
+</joint>
 <!-- ............................. CAMERA ........................................ -->
 <xacro:if value="$(arg camera_enabled)">

Commit message: Updated chassis with logo, readme, imu

File: urdf/gazebo.xacro (robot description, xacro)
@@ -29,29 +29,14 @@
 </gazebo>
 <!--............................... IMU PLUGIN ..................................... -->
-<!-- <gazebo>
-	<plugin name="imu_plugin" filename="libgazebo_ros_imu.so">
-		<updateRate>50.0</updateRate>
-		<robotNamespace>$(arg robot_namespace)</robotNamespace>
-		<bodyName>base_link</bodyName>
-		<topicName>/imu</topicName>
-		<serviceName>/imu/calibrate</serviceName>
-		<accelOffset>0.0 0.0 0.0</accelOffset>
-		<accelDrift>0.0 0.0 0.0</accelDrift>
-		<accelDriftFrequency>0.0 0.0 0.0</accelDriftFrequency>
-		<accelGaussianNoise>0.0 0.0 0.0</accelGaussianNoise>
-		<rateOffset>0.0 0.0 0.0</rateOffset>
-		<rateDrift>0.0 0.0 0.0</rateDrift>
-		<rateDriftFrequency>0.0 0.0 0.0</rateDriftFrequency>
-		<rateGaussianNoise>0.0 0.0 0.0</rateGaussianNoise>
-		<headingOffset>0.0</headingOffset>
-		<headingDrift>0.0</headingDrift>
-		<headingDriftFrequency>0.0</headingDriftFrequency>
-		<headingGaussianNoise>0.0</headingGaussianNoise>
-		<rpyOffset>0.0 0.0 0.0</rpyOffset>
-		<xyzOffset>0.0 0.0 0.0</xyzOffset>
-		<gaussianNoise>0.0</gaussianNoise>
-		<frameName>imu_frame</frameName>
-	</plugin>
-</gazebo> -->
+<gazebo reference="imu_frame">
+	<sensor name="my_imu" type="imu">
+    <always_on>true</always_on>
+    <plugin name="my_imu_plugin" filename="libgazebo_ros_imu_sensor.so">
+      <topicName>$(arg robot_namespace)/imu</topicName>
+      <updateRate>5</updateRate>
+      <frameName>imu_frame</frameName>
+    </plugin>
+  </sensor>
+</gazebo>
 <!--............................... Ground truth PLUGIN .............................-->
 <gazebo>

File: urdf/new_bcr_robot.xacro (robot description, xacro)
@@ -102,4 +102,11 @@
    </gazebo>
 </xacro:if>
+<!-- ............................. IMU ........................................ -->
+<link name="imu_frame"/>
+<joint name="imu_joint" type="fixed">
+    <parent link="base_link"/>
+    <child link="imu_frame"/>
+    <origin xyz="0.0 0.0 0.08" rpy="0.0 0.0 0.0"/>
+</joint>
 <!-- ............................. CAMERA ........................................ -->
 <xacro:if value="$(arg camera_enabled)">
