Commit message: updated readme

File: urdf/bcr_bot.xacro (robot description, xacro)
@@ -1,4 +1,4 @@
 <?xml version="1.0"?>
-<robot xmlns:xacro="http://www.ros.org/wiki/xacro" name="new_bcr_robot">
+<robot xmlns:xacro="http://www.ros.org/wiki/xacro" name="bcr_bot">
 <!--................................ XACRO CONSTANTS .............................. -->
 <xacro:property name="chassis_mass"                value="70"/>
@@ -28,5 +28,5 @@
 <xacro:property name="camera_height"               value="0.10"/>
 <xacro:property name="camera_horizontal_fov"       value="60"/>
-<xacro:arg      name="robot_namespace"             default="new_bcr_robot"/>
+<xacro:arg      name="robot_namespace"             default="bcr_bot"/>
 <xacro:arg      name="wheel_odom_topic"            default="odom" />
 <xacro:arg      name="camera_enabled"              default="false" />
@@ -38,11 +38,11 @@
 <xacro:arg      name="sim_gz"                      default="false" />
 <!-- ............................... LOAD MACROS ................................. -->
-<xacro:include filename="$(find new_bcr_robot)/urdf/materials.xacro"/>
-<xacro:include filename="$(find new_bcr_robot)/urdf/macros.xacro"/>
+<xacro:include filename="$(find bcr_bot)/urdf/materials.xacro"/>
+<xacro:include filename="$(find bcr_bot)/urdf/macros.xacro"/>
 <xacro:if value="$(arg sim_gazebo)">
-	<xacro:include filename="$(find new_bcr_robot)/urdf/gazebo.xacro"/>
+	<xacro:include filename="$(find bcr_bot)/urdf/gazebo.xacro"/>
 </xacro:if>
 <xacro:if value="$(arg sim_gz)">
-	<xacro:include filename="$(find new_bcr_robot)/urdf/gz.xacro"/>
+	<xacro:include filename="$(find bcr_bot)/urdf/gz.xacro"/>
 </xacro:if>
 <!-- ................................ BASE LINK .................................. -->
@@ -58,5 +58,5 @@
 		<origin xyz="0 0 -0.205" rpy="0 0 0" />
   		<geometry>
-    		<mesh filename="file://$(find new_bcr_robot)/meshes/bcr_bot_mesh.dae" scale="1 1 1"/>
+    		<mesh filename="file://$(find bcr_bot)/meshes/bcr_bot_mesh.dae" scale="1 1 1"/>
   		</geometry>
 	</visual>
@@ -129,5 +129,5 @@
 			<origin xyz="0 0 0" rpy="0 0 0" />
 				<geometry>
-					<mesh filename="file://$(find new_bcr_robot)/meshes/kinect/d415.dae"/>
+					<mesh filename="file://$(find bcr_bot)/meshes/kinect/d415.dae"/>
 				</geometry>
 				<material name="black"/>

File: urdf/gazebo.xacro (robot description, xacro)
@@ -1,4 +1,4 @@
 <?xml version="1.0"?>
-<robot xmlns:xacro="http://www.ros.org/wiki/xacro" name="new_bcr_robot">
+<robot xmlns:xacro="http://www.ros.org/wiki/xacro" name="bcr_bot">
 <gazebo>
 	<static>false</static>

File: urdf/gz.xacro (robot description, xacro)
@@ -1,4 +1,4 @@
 <?xml version="1.0"?>
-<robot xmlns:xacro="http://www.ros.org/wiki/xacro" name="new_bcr_robot">
+<robot xmlns:xacro="http://www.ros.org/wiki/xacro" name="bcr_bot">
 <!-- ........................... SENSOR PLUGIN ................................... -->
 <gazebo>

File: urdf/macros.xacro (robot description, xacro)
@@ -1,4 +1,4 @@
 <?xml version="1.0"?>
-<robot xmlns:xacro="http://www.ros.org/wiki/xacro" name="new_bcr_robot">
+<robot xmlns:xacro="http://www.ros.org/wiki/xacro" name="bcr_bot">
 <!--................................ INERTIA MATRICES .............................. -->
 <xacro:macro name="cylinder_inertia" params="m r h">

File: urdf/materials.xacro (robot description, xacro)
@@ -1,4 +1,4 @@
 <?xml version="1.0"?>
-<robot xmlns:xacro="http://www.ros.org/wiki/xacro" name="new_bcr_robot">
+<robot xmlns:xacro="http://www.ros.org/wiki/xacro" name="bcr_bot">
 	<material name="black">
 		<color rgba="0.0 0.0 0.0 1.0"/>

Commit message: updated readme

File: urdf/bcr_bot.xacro (robot description, xacro)
@@ -1,4 +1,4 @@
 <?xml version="1.0"?>
-<robot xmlns:xacro="http://www.ros.org/wiki/xacro" name="new_bcr_robot">
+<robot xmlns:xacro="http://www.ros.org/wiki/xacro" name="bcr_bot">
 <!--................................ XACRO CONSTANTS .............................. -->
 <xacro:property name="chassis_mass"                value="70"/>
@@ -36,7 +36,7 @@
 <xacro:arg      name="ground_truth_frame"          default="map"/>
 <!-- ............................... LOAD MACROS ................................. -->
-<xacro:include filename="$(find new_bcr_robot)/urdf/materials.xacro"/>
-<xacro:include filename="$(find new_bcr_robot)/urdf/macros.xacro"/>
-<xacro:include filename="$(find new_bcr_robot)/urdf/gazebo.xacro"/>
+<xacro:include filename="$(find bcr_bot)/urdf/materials.xacro"/>
+<xacro:include filename="$(find bcr_bot)/urdf/macros.xacro"/>
+<xacro:include filename="$(find bcr_bot)/urdf/gazebo.xacro"/>
 <!-- ................................ BASE LINK .................................. -->
 <link name="base_link"/>
@@ -51,5 +51,5 @@
 		<origin xyz="0 0 -0.2" rpy="0 0 0" />
   		<geometry>
-    		<mesh filename="file://$(find new_bcr_robot)/meshes/bcr_bot_mesh.dae" scale="1 1 1"/>
+    		<mesh filename="file://$(find bcr_bot)/meshes/bcr_bot_mesh.dae" scale="1 1 1"/>
   		</geometry>
 	</visual>
@@ -122,5 +122,5 @@
 			<origin xyz="0 0 0" rpy="0 0 0" />
 				<geometry>
-					<mesh filename="file://$(find new_bcr_robot)/meshes/kinect/d415.dae"/>
+					<mesh filename="file://$(find bcr_bot)/meshes/kinect/d415.dae"/>
 				</geometry>
 				<material name="black"/>

File: urdf/gazebo.xacro (robot description, xacro)
@@ -1,4 +1,4 @@
 <?xml version="1.0"?>
-<robot xmlns:xacro="http://www.ros.org/wiki/xacro" name="new_bcr_robot">
+<robot xmlns:xacro="http://www.ros.org/wiki/xacro" name="bcr_bot">
 <gazebo>
   <static>false</static>

File: urdf/macros.xacro (robot description, xacro)
@@ -1,4 +1,4 @@
 <?xml version="1.0"?>
-<robot xmlns:xacro="http://www.ros.org/wiki/xacro" name="new_bcr_robot">
+<robot xmlns:xacro="http://www.ros.org/wiki/xacro" name="bcr_bot">
 <!--................................ INERTIA MATRICES .............................. -->
 <xacro:macro name="cylinder_inertia" params="m r h">

File: urdf/materials.xacro (robot description, xacro)
@@ -1,4 +1,4 @@
 <?xml version="1.0"?>
-<robot xmlns:xacro="http://www.ros.org/wiki/xacro" name="new_bcr_robot">
+<robot xmlns:xacro="http://www.ros.org/wiki/xacro" name="bcr_bot">
 <material name="black">
 	<color rgba="0.0 0.0 0.0 1.0"/>

Commit message: namespace-fix

File: urdf/bcr_bot.xacro (robot description, xacro)
@@ -23,5 +23,5 @@
 <xacro:property name="two_d_lidar_min_angle"       value="0"/>
 <xacro:property name="two_d_lidar_max_angle"       value="360"/>
-<xacro:property name="two_d_lidar_min_range"       value="0.1"/>
+<xacro:property name="two_d_lidar_min_range"       value="0.55"/>
 <xacro:property name="two_d_lidar_max_range"       value="16"/>
 <xacro:property name="camera_baseline"             value="0.06"/>
@@ -35,4 +35,5 @@
 <xacro:arg      name="conveyor_enabled"            default="false"/>
 <xacro:arg      name="ground_truth_frame"          default="map"/>
+<xacro:arg      name="odometry_source"             default="world"/>
 <!-- ............................... LOAD MACROS ................................. -->
 <xacro:include filename="$(find bcr_bot)/urdf/materials.xacro"/>
@@ -96,5 +97,5 @@
       <parent link="base_link"/>
       <child link="two_d_lidar"/>
-      <origin xyz="0.3 0 0.08" rpy="0 0 0" />
+      <origin xyz="0 0 0.08" rpy="0 0 0" />
     </joint>
    <gazebo reference="two_d_lidar">

File: urdf/gazebo.xacro (robot description, xacro)
@@ -24,5 +24,5 @@
 		<publishWheelJointState>true</publishWheelJointState>
 		<publishOdometryMsg>true</publishOdometryMsg>
-		<odometrySource>encoder</odometrySource>
+		<odometrySource>$(arg odometry_source)</odometrySource>
 		<wheelAcceleration>5.0</wheelAcceleration>
 	</plugin>

Commit message: fixed namespace updated readme

File: urdf/bcr_bot.xacro (robot description, xacro)
@@ -23,5 +23,5 @@
 <xacro:property name="two_d_lidar_min_angle"       value="0"/>
 <xacro:property name="two_d_lidar_max_angle"       value="360"/>
-<xacro:property name="two_d_lidar_min_range"       value="0.1"/>
+<xacro:property name="two_d_lidar_min_range"       value="0.55"/>
 <xacro:property name="two_d_lidar_max_range"       value="16"/>
 <xacro:property name="camera_baseline"             value="0.06"/>
@@ -37,4 +37,6 @@
 <xacro:arg      name="sim_gazebo"                  default="false" />
 <xacro:arg      name="sim_gz"                      default="false" />
+<xacro:arg      name="odometry_source"             default="world" />
+<xacro:property name="odometry_source"             value="$(arg odometry_source)"/>
 <!-- ............................... LOAD MACROS ................................. -->
 <xacro:include filename="$(find bcr_bot)/urdf/materials.xacro"/>
@@ -103,5 +105,5 @@
       <parent link="base_link"/>
       <child link="two_d_lidar"/>
-      <origin xyz="0.3 0 0.08" rpy="0 0 0" />
+      <origin xyz="0.0 0 0.08" rpy="0 0 0" />
     </joint>
    <gazebo reference="two_d_lidar">

File: urdf/gazebo.xacro (robot description, xacro)
@@ -27,4 +27,11 @@
 		<publish_odom>true</publish_odom>
 		<max_wheel_acceleration>5.0</max_wheel_acceleration>
+		<!-- Odometry source, 0 for ENCODER, 1 for WORLD, defaults to WORLD -->
+		<xacro:if value="${odometry_source == 'world'}">
+			<odometry_source>1</odometry_source>
+		</xacro:if>
+		<xacro:if value="${odometry_source == 'encoder'}">
+			<odometry_source>0</odometry_source>
+		</xacro:if>
 	</plugin>
 </gazebo>
@@ -90,5 +97,5 @@
 				</ros>
 				<output_type>sensor_msgs/LaserScan</output_type>
-				<frameName>two_d_lidar</frameName>
+				<frame_name>two_d_lidar</frame_name>
 			</plugin>
 		</sensor>

File: urdf/gz.xacro (robot description, xacro)
@@ -8,4 +8,7 @@
     <plugin filename="ignition-gazebo-imu-system"
         name="ignition::gazebo::systems::Imu">
+    </plugin>
+    <plugin filename="ignition-gazebo-joint-state-publisher-system"
+        name="ignition::gazebo::systems::JointStatePublisher">
     </plugin>
 <!-- ........................... DIFFERENTIAL DRIVE PLUGIN ................................... -->
@@ -60,5 +63,5 @@
         <sensor type="depth_camera" name="kinect_camera">
             <update_rate>30.0</update_rate>
-            <topic>depth_camera</topic>
+            <topic>kinect_camera</topic>
             <ignition_frame_id>kinect_camera</ignition_frame_id>
             <camera_info_topic>camera_info</camera_info_topic>

Commit message: overwritten parameters fixed

File: urdf/bcr_bot.xacro (robot description, xacro)
@@ -11,5 +11,5 @@
 <xacro:property name="traction_wheel_friction"     value="5.0"/>
 <xacro:property name="trolley_wheel_mass"          value="0.1"/>
-<xacro:property name="trolley_wheel_base"          value="0.54"/>
+<xacro:property name="trolley_track_width"          value="0.54"/>
 <xacro:property name="trolley_wheel_friction"      value="0.0"/>
 <xacro:property name="trolley_wheel_radius"        value="0.06"/>
@@ -18,5 +18,5 @@
 <xacro:property name="traction_wheel_radius"       value="0.1"/>
 <xacro:property name="traction_wheel_width"        value="0.05"/>
-<xacro:property name="traction_wheel_base"         value="0.8"/>
+<xacro:property name="traction_track_width"         value="0.8"/>
 <xacro:property name="two_d_lidar_update_rate"     value="30"/>
 <xacro:property name="two_d_lidar_sample_size"     value="361"/>
@@ -74,10 +74,10 @@
 </joint>
 <!-- ................................ WHEELS ..................................... -->
-<xacro:trolley_wheel cardinality="front" dexterity="left"  origin_x="${chassis_length/2}" origin_y="${trolley_wheel_base/2}" origin_z="-${trolley_wheel_radius+chassis_height/2}"/>
-<xacro:trolley_wheel cardinality="front" dexterity="right" origin_x="${chassis_length/2}" origin_y="-${trolley_wheel_base/2}" origin_z="-${trolley_wheel_radius+chassis_height/2}"/>
-<xacro:trolley_wheel cardinality="back" dexterity="left"  origin_x="-${chassis_length/2}" origin_y="${trolley_wheel_base/2}" origin_z="-${trolley_wheel_radius+chassis_height/2}"/>
-<xacro:trolley_wheel cardinality="back" dexterity="right" origin_x="-${chassis_length/2}" origin_y="-${trolley_wheel_base/2}" origin_z="-${trolley_wheel_radius+chassis_height/2}"/>
-<xacro:traction_wheel cardinality="middle" dexterity="left"  origin_x="0" origin_y="${traction_wheel_base/2}" origin_z="-${chassis_height/2+2*trolley_wheel_radius+eps-traction_wheel_radius}"/>
-<xacro:traction_wheel cardinality="middle" dexterity="right" origin_x="0" origin_y="-${traction_wheel_base/2}" origin_z="-${chassis_height/2+2*trolley_wheel_radius+eps-traction_wheel_radius}"/>
+<xacro:trolley_wheel cardinality="front" dexterity="left"  origin_x="${chassis_length/2}" origin_y="${trolley_track_width/2}" origin_z="-${trolley_wheel_radius+chassis_height/2}"/>
+<xacro:trolley_wheel cardinality="front" dexterity="right" origin_x="${chassis_length/2}" origin_y="-${trolley_track_width/2}" origin_z="-${trolley_wheel_radius+chassis_height/2}"/>
+<xacro:trolley_wheel cardinality="back" dexterity="left"  origin_x="-${chassis_length/2}" origin_y="${trolley_track_width/2}" origin_z="-${trolley_wheel_radius+chassis_height/2}"/>
+<xacro:trolley_wheel cardinality="back" dexterity="right" origin_x="-${chassis_length/2}" origin_y="-${trolley_track_width/2}" origin_z="-${trolley_wheel_radius+chassis_height/2}"/>
+<xacro:traction_wheel cardinality="middle" dexterity="left"  origin_x="0" origin_y="${traction_track_width/2}" origin_z="-${chassis_height/2+2*trolley_wheel_radius+eps-traction_wheel_radius}"/>
+<xacro:traction_wheel cardinality="middle" dexterity="right" origin_x="0" origin_y="-${traction_track_width/2}" origin_z="-${chassis_height/2+2*trolley_wheel_radius+eps-traction_wheel_radius}"/>
 <!-- ............................. 2D LIDAR ........................................ -->
 <xacro:if value="$(arg two_d_lidar_enabled)">

File: urdf/gazebo.xacro (robot description, xacro)
@@ -16,5 +16,5 @@
 		<left_joint>middle_left_wheel_joint</left_joint>
 		<right_joint>middle_right_wheel_joint</right_joint>
-		<wheel_separation>${traction_wheel_base+traction_wheel_width-0.01}</wheel_separation>
+		<wheel_separation>${traction_track_width+traction_wheel_width-0.01}</wheel_separation>
 		<wheel_diameter>${2*traction_wheel_radius+0.01}</wheel_diameter>
 		<robot_base_frame>base_link</robot_base_frame>

File: urdf/gz.xacro (robot description, xacro)
@@ -16,5 +16,5 @@
         <left_joint>middle_left_wheel_joint</left_joint>
         <right_joint>middle_right_wheel_joint</right_joint>
-        <wheel_separation>${traction_wheel_base+traction_wheel_width-0.01}</wheel_separation>
+        <wheel_separation>${traction_track_width+traction_wheel_width-0.01}</wheel_separation>
         <wheel_radius>${traction_wheel_radius+0.01}</wheel_radius>
         <odom_publish_frequency>30</odom_publish_frequency>

Commit message: fixed overwritten parameters

File: urdf/bcr_bot.xacro (robot description, xacro)
@@ -11,5 +11,5 @@
 <xacro:property name="traction_wheel_friction"     value="5.0"/>
 <xacro:property name="trolley_wheel_mass"          value="0.1"/>
-<xacro:property name="trolley_wheel_base"          value="0.54"/>
+<xacro:property name="trolley_track_width"          value="0.54"/>
 <xacro:property name="trolley_wheel_friction"      value="0.0"/>
 <xacro:property name="trolley_wheel_radius"        value="0.06"/>
@@ -18,5 +18,5 @@
 <xacro:property name="traction_wheel_radius"       value="0.1"/>
 <xacro:property name="traction_wheel_width"        value="0.05"/>
-<xacro:property name="traction_wheel_base"         value="0.8"/>
+<xacro:property name="traction_track_width"         value="0.8"/>
 <xacro:property name="two_d_lidar_update_rate"     value="30"/>
 <xacro:property name="two_d_lidar_sample_size"     value="361"/>
@@ -66,10 +66,10 @@
 </joint>
 <!-- ................................ WHEELS ..................................... -->
-<xacro:trolley_wheel cardinality="front" dexterity="left"  origin_x="${chassis_length/2}" origin_y="${trolley_wheel_base/2}" origin_z="-${trolley_wheel_radius+chassis_height/2}"/>
-<xacro:trolley_wheel cardinality="front" dexterity="right" origin_x="${chassis_length/2}" origin_y="-${trolley_wheel_base/2}" origin_z="-${trolley_wheel_radius+chassis_height/2}"/>
-<xacro:trolley_wheel cardinality="back" dexterity="left"  origin_x="-${chassis_length/2}" origin_y="${trolley_wheel_base/2}" origin_z="-${trolley_wheel_radius+chassis_height/2}"/>
-<xacro:trolley_wheel cardinality="back" dexterity="right" origin_x="-${chassis_length/2}" origin_y="-${trolley_wheel_base/2}" origin_z="-${trolley_wheel_radius+chassis_height/2}"/>
-<xacro:traction_wheel cardinality="middle" dexterity="left"  origin_x="0" origin_y="${traction_wheel_base/2}" origin_z="-${chassis_height/2+2*trolley_wheel_radius+eps-traction_wheel_radius}"/>
-<xacro:traction_wheel cardinality="middle" dexterity="right" origin_x="0" origin_y="-${traction_wheel_base/2}" origin_z="-${chassis_height/2+2*trolley_wheel_radius+eps-traction_wheel_radius}"/>
+<xacro:trolley_wheel cardinality="front" dexterity="left"  origin_x="${chassis_length/2}" origin_y="${trolley_track_width/2}" origin_z="-${trolley_wheel_radius+chassis_height/2}"/>
+<xacro:trolley_wheel cardinality="front" dexterity="right" origin_x="${chassis_length/2}" origin_y="-${trolley_track_width/2}" origin_z="-${trolley_wheel_radius+chassis_height/2}"/>
+<xacro:trolley_wheel cardinality="back" dexterity="left"  origin_x="-${chassis_length/2}" origin_y="${trolley_track_width/2}" origin_z="-${trolley_wheel_radius+chassis_height/2}"/>
+<xacro:trolley_wheel cardinality="back" dexterity="right" origin_x="-${chassis_length/2}" origin_y="-${trolley_track_width/2}" origin_z="-${trolley_wheel_radius+chassis_height/2}"/>
+<xacro:traction_wheel cardinality="middle" dexterity="left"  origin_x="0" origin_y="${traction_track_width/2}" origin_z="-${chassis_height/2+2*trolley_wheel_radius+eps-traction_wheel_radius}"/>
+<xacro:traction_wheel cardinality="middle" dexterity="right" origin_x="0" origin_y="-${traction_track_width/2}" origin_z="-${chassis_height/2+2*trolley_wheel_radius+eps-traction_wheel_radius}"/>
 <!-- ............................. 2D LIDAR ........................................ -->
 <xacro:if value="$(arg two_d_lidar_enabled)">

File: urdf/gazebo.xacro (robot description, xacro)
@@ -12,5 +12,5 @@
 		<leftJoint>middle_left_wheel_joint</leftJoint>
 		<rightJoint>middle_right_wheel_joint</rightJoint>
-		<wheelSeparation>${traction_wheel_base+traction_wheel_width-0.01}</wheelSeparation>
+		<wheelSeparation>${traction_track_width+traction_wheel_width-0.01}</wheelSeparation>
 		<wheelDiameter>${2*traction_wheel_radius+0.01}</wheelDiameter>
 		<robotBaseFrame>base_link</robotBaseFrame>
