Commit message: added stereo_cam to bcr_bot

File: urdf/bcr_bot.xacro (robot description, xacro)
@@ -31,4 +31,5 @@
 <xacro:arg      name="wheel_odom_topic"            default="odom" />
 <xacro:arg      name="camera_enabled"              default="false" />
+<xacro:arg      name="stereo_camera_enabled"       default="false" />
 <xacro:arg      name="two_d_lidar_enabled"         default="false" />
 <xacro:arg      name="publish_wheel_odom_tf"       default="true" />
@@ -152,4 +153,38 @@
 	</joint>
 </xacro:if>
+<!-- .............................STEREO CAMERA ........................................ -->
+<xacro:if value="$(arg stereo_camera_enabled)">
+	<!-- STEREO CAMERA -->
+	<link name="stereo_camera">
+		<collision>
+			<origin xyz="0 0 0" rpy="0 0 0" />
+				<geometry>
+					<box size="0.07 0.3 0.09"/>
+				</geometry>
+		</collision>
+		<visual>
+			<origin xyz="0 0 0" rpy="0 0 0" />
+				<geometry>
+					<mesh filename="file://$(find bcr_bot)/meshes/kinect/d415.dae"/>
+				</geometry>
+				<material name="black"/>
+		</visual>
+		<inertial>
+				<mass value="0.01"/>
+				<xacro:box_inertia m="0.01" x="0.07" y="0.3" z = "0.09"/>
+		</inertial>
+	</link>
+	<joint name="stereo_camera_joint" type="fixed">
+			<origin rpy="0 0 0" xyz="${chassis_length/2} 0 ${chassis_height/7}"/>
+			<parent link="base_link"/>
+			<child link="stereo_camera"/>
+	</joint>
+	<link name="stereo_camera_optical"/>
+	<joint name="stereo_camera_optical_joint" type="fixed">
+		<origin xyz="0 0 0" rpy="${-pi/2} 0 ${-pi/2}"/>
+		<parent link="stereo_camera"/>
+		<child link="stereo_camera_optical"/>
+	</joint>
+</xacro:if>
 <!-- ............................. ROOF ........................................ -->
 <link name="roof_link">

File: urdf/gazebo.xacro (robot description, xacro)
@@ -132,4 +132,74 @@
 	</gazebo>
 </xacro:if>
-<!--................................................................................. -->
+<!-- ...........................STEREO CAMERA PLUGIN ................................... -->
+<xacro:if value="$(arg stereo_camera_enabled)">
+	<gazebo reference="stereo_camera">
+		<sensor type="multicamera" name="stereo_camera">
+			<update_rate>10.0</update_rate>
+			<always_on>true</always_on>
+			<camera name="left">
+				<pose>0 0 0 0 0 0</pose>
+				<horizontal_fov>1.3962634</horizontal_fov>
+				<image>
+				<width>1024</width>
+				<height>1024</height>
+				<format>R8G8B8</format>
+				</image>
+				<clip>
+				<near>0.3</near>
+				<far>20</far>
+				</clip>
+				<noise>
+				<type>gaussian</type>
+				<mean>0.0</mean>
+				<stddev>0.0</stddev>
+				</noise>
+				<distortion>
+				<k1>0.0</k1>
+				<k2>0.0</k2>
+				<k3>0.0</k3>
+				<p1>0.0</p1>
+				<p2>0.0</p2>
+				<center>0.5 0.5</center>
+				</distortion>
+			</camera>
+			<camera name="right">
+				<pose>0 -0.12 0 0 0 0</pose>
+				<horizontal_fov>1.3962634</horizontal_fov>
+				<image>
+				<width>1024</width>
+				<height>1024</height>
+				<format>R8G8B8</format>
+				</image>
+				<clip>
+				<near>0.3</near>
+				<far>20</far>
+				</clip>
+				<noise>
+				<type>gaussian</type>
+				<mean>0.0</mean>
+				<stddev>0.0</stddev>
+				</noise>
+				<distortion>
+				<k1>0.0</k1>
+				<k2>0.0</k2>
+				<k3>0.0</k3>
+				<p1>0.0</p1>
+				<p2>0.0</p2>
+				<center>0.5 0.5</center>
+				</distortion>
+			</camera>
+			<plugin name="stereo_camera_controller" filename="libgazebo_ros_camera.so">
+				<ros>
+				<namespace>$(arg robot_namespace)</namespace>
+				<argument>image_raw:=image_raw</argument>
+				<argument>camera_info:=camera_info</argument>
+				</ros>
+				<camera_name>stereo_camera</camera_name>
+				<frame_name>stereo_camera_optical</frame_name>
+				<hack_baseline>0.12</hack_baseline>
+			</plugin>
+		</sensor>
+	</gazebo>
+</xacro:if>
 </robot>

File: urdf/gz.xacro (robot description, xacro)
@@ -3,91 +3,132 @@
 <!-- ........................... SENSOR PLUGIN ................................... -->
 <gazebo>
-    <plugin filename="ignition-gazebo-sensors-system" name="ignition::gazebo::systems::Sensors">
-        <render_engine>ogre2</render_engine>
-    </plugin>
-    <plugin filename="ignition-gazebo-imu-system"
-        name="ignition::gazebo::systems::Imu">
-    </plugin>
-    <plugin filename="ignition-gazebo-joint-state-publisher-system"
-        name="ignition::gazebo::systems::JointStatePublisher">
-    </plugin>
+	<plugin filename="ignition-gazebo-sensors-system" name="ignition::gazebo::systems::Sensors">
+		<render_engine>ogre2</render_engine>
+	</plugin>
+	<plugin filename="ignition-gazebo-imu-system"
+		name="ignition::gazebo::systems::Imu">
+	</plugin>
+	<plugin filename="ignition-gazebo-joint-state-publisher-system"
+		name="ignition::gazebo::systems::JointStatePublisher">
+	</plugin>
 <!-- ........................... DIFFERENTIAL DRIVE PLUGIN ................................... -->
-    <plugin filename="ignition-gazebo-diff-drive-system" name="ignition::gazebo::systems::DiffDrive">
-        <left_joint>middle_left_wheel_joint</left_joint>
-        <right_joint>middle_right_wheel_joint</right_joint>
-        <wheel_separation>${traction_track_width+traction_wheel_width-0.01}</wheel_separation>
-        <wheel_radius>${traction_wheel_radius+0.01}</wheel_radius>
-        <odom_publish_frequency>30</odom_publish_frequency>
-        <topic>/cmd_vel</topic>
-        <odom_topic>$(arg wheel_odom_topic)</odom_topic>
-        <tf_topic>/tf</tf_topic>
-        <frame_id>odom</frame_id>
-        <child_frame_id>base_link</child_frame_id>
-    </plugin>
+	<plugin filename="ignition-gazebo-diff-drive-system" name="ignition::gazebo::systems::DiffDrive">
+		<left_joint>middle_left_wheel_joint</left_joint>
+		<right_joint>middle_right_wheel_joint</right_joint>
+		<wheel_separation>${traction_track_width+traction_wheel_width-0.01}</wheel_separation>
+		<wheel_radius>${traction_wheel_radius+0.01}</wheel_radius>
+		<odom_publish_frequency>30</odom_publish_frequency>
+		<topic>/cmd_vel</topic>
+		<odom_topic>$(arg wheel_odom_topic)</odom_topic>
+		<tf_topic>/tf</tf_topic>
+		<frame_id>odom</frame_id>
+		<child_frame_id>base_link</child_frame_id>
+	</plugin>
 </gazebo>
 <!-- ........................... 2D LIDAR config ................................... -->
 <xacro:if value="$(arg two_d_lidar_enabled)">
-    <gazebo reference="two_d_lidar">
-        <sensor name='gpu_lidar' type='gpu_lidar'>
-            <topic>scan</topic>
-            <update_rate>${two_d_lidar_update_rate}</update_rate>
-            <ignition_frame_id>two_d_lidar</ignition_frame_id>
-            <lidar>
-                <scan>
-                    <horizontal>
-                        <samples>${two_d_lidar_sample_size}</samples>
-                        <resolution>1</resolution>
-                        <min_angle>${radians(two_d_lidar_min_angle)}</min_angle>
-                        <max_angle>${radians(two_d_lidar_max_angle)}</max_angle>
-                    </horizontal>
-                </scan>
-                <range>
-                    <min>${two_d_lidar_min_range}</min>
-                    <max>${two_d_lidar_max_range}</max>
-                    <resolution>0.01</resolution>
-                </range>
-                <noise>
-                    <type>gaussian</type>
-                    <mean>0.0</mean>
-                    <stddev>0.001</stddev>
-                </noise>
-            </lidar>
-            <alwaysOn>1</alwaysOn>
-            <visualize>true</visualize>
-        </sensor>
-    </gazebo>
+	<gazebo reference="two_d_lidar">
+		<sensor name='gpu_lidar' type='gpu_lidar'>
+			<topic>scan</topic>
+			<update_rate>${two_d_lidar_update_rate}</update_rate>
+			<ignition_frame_id>two_d_lidar</ignition_frame_id>
+			<lidar>
+				<scan>
+					<horizontal>
+						<samples>${two_d_lidar_sample_size}</samples>
+						<resolution>1</resolution>
+						<min_angle>${radians(two_d_lidar_min_angle)}</min_angle>
+						<max_angle>${radians(two_d_lidar_max_angle)}</max_angle>
+					</horizontal>
+				</scan>
+				<range>
+					<min>${two_d_lidar_min_range}</min>
+					<max>${two_d_lidar_max_range}</max>
+					<resolution>0.01</resolution>
+				</range>
+				<noise>
+					<type>gaussian</type>
+					<mean>0.0</mean>
+					<stddev>0.001</stddev>
+				</noise>
+			</lidar>
+			<alwaysOn>1</alwaysOn>
+			<visualize>true</visualize>
+		</sensor>
+	</gazebo>
 </xacro:if>
 <!-- ........................... CAMERA config ................................... -->
 <xacro:if value="$(arg camera_enabled)">
-    <gazebo reference="kinect_camera">
-        <sensor type="depth_camera" name="kinect_camera">
-            <update_rate>30.0</update_rate>
-            <topic>kinect_camera</topic>
-            <ignition_frame_id>kinect_camera</ignition_frame_id>
-            <camera_info_topic>camera_info</camera_info_topic>
-            <camera>
-                <horizontal_fov>${radians(camera_horizontal_fov)}</horizontal_fov>
-                <image>
-                    <width>640</width>
-                    <height>480</height>
-                    <format>R8G8B8</format>
-                </image>
-                <clip>
-                    <near>0.05</near>
-                    <far>8.0</far>
-                </clip>
-            </camera>
-        </sensor>
-    </gazebo>
+	<gazebo reference="kinect_camera">
+		<sensor type="depth_camera" name="kinect_camera">
+			<update_rate>30.0</update_rate>
+			<topic>kinect_camera</topic>
+			<ignition_frame_id>kinect_camera</ignition_frame_id>
+			<camera_info_topic>kinect_camera/camera_info</camera_info_topic>
+			<camera>
+				<horizontal_fov>${radians(camera_horizontal_fov)}</horizontal_fov>
+				<image>
+					<width>640</width>
+					<height>480</height>
+					<format>R8G8B8</format>
+				</image>
+				<clip>
+					<near>0.05</near>
+					<far>8.0</far>
+				</clip>
+			</camera>
+		</sensor>
+	</gazebo>
 </xacro:if>
 <!-- ........................... IMU config ................................... -->
 <gazebo reference="imu_frame">
-    <sensor name="imu_sensor" type="imu">
-        <always_on>1</always_on>
-        <update_rate>1</update_rate>
-        <ignition_frame_id>imu_frame</ignition_frame_id>
-        <visualize>true</visualize>
-        <topic>imu</topic>
-    </sensor>
+	<sensor name="imu_sensor" type="imu">
+		<always_on>1</always_on>
+		<update_rate>1</update_rate>
+		<ignition_frame_id>imu_frame</ignition_frame_id>
+		<visualize>true</visualize>
+		<topic>imu</topic>
+	</sensor>
 </gazebo>
+<!-- ........................... Stereo camera ................................... -->
+<xacro:if value="$(arg stereo_camera_enabled)">
+	<gazebo reference="stereo_camera">
+		<sensor type="camera" name="right">
+			<update_rate>10.0</update_rate>
+			<always_on>true</always_on>
+			<ignition_frame_id>stereo_camera_optical</ignition_frame_id>
+			<pose>0 -0.12 0 0 0 0</pose>
+			<topic>stereo_camera/right/image_raw</topic>
+			<camera_info_topic>stereo_camera/right/camera_info</camera_info_topic>
+			<horizontal_fov>1.3962634</horizontal_fov>
+			<image>
+				<width>1024</width>
+				<height>1024</height>
+				<format>R8G8B8</format>
+			</image>
+			<clip>
+				<near>0.3</near>
+				<far>20</far>
+			</clip>
+		</sensor>
+		<sensor type="camera" name="left">
+			<topic>stereo_camera/left/image_raw</topic>
+			<update_rate>10.0</update_rate>
+			<always_on>true</always_on>
+			<ignition_frame_id>stereo_camera_optical</ignition_frame_id>
+			<camera_info_topic>stereo_camera/left/camera_info</camera_info_topic>
+			<pose>0 0 0 0 0 0</pose>
+			<horizontal_fov>1.3962634</horizontal_fov>
+			<image>
+				<width>1024</width>
+				<height>1024</height>
+				<format>R8G8B8</format>
+			</image>
+			<clip>
+				<near>0.3</near>
+				<far>20</far>
+			</clip>
+		</sensor>
+	</gazebo>
+</xacro:if>
 </robot>

Commit message: added stereo camera

File: urdf/bcr_bot.xacro (robot description, xacro)
@@ -31,4 +31,5 @@
 <xacro:arg      name="wheel_odom_topic"            default="odom"/>
 <xacro:arg      name="camera_enabled"              default="false"/>
+<xacro:arg      name="stereo_camera_enabled"       default="false" />
 <xacro:arg      name="two_d_lidar_enabled"         default="false"/>
 <xacro:arg      name="publish_wheel_odom_tf"       default="true"/>
@@ -144,4 +145,38 @@
 	</joint>
 </xacro:if>
+<!-- .............................. STEREO CAMERA ........................................ -->
+<xacro:if value="$(arg stereo_camera_enabled)">
+	<!-- STEREO CAMERA -->
+	<link name="stereo_camera">
+		<collision>
+			<origin xyz="0 0 0" rpy="0 0 0" />
+				<geometry>
+					<box size="0.07 0.3 0.09"/>
+				</geometry>
+		</collision>
+		<visual>
+			<origin xyz="0 0 0" rpy="0 0 0" />
+				<geometry>
+					<mesh filename="file://$(find bcr_bot)/meshes/kinect/d415.dae"/>
+				</geometry>
+				<material name="black"/>
+		</visual>
+		<inertial>
+				<mass value="0.01"/>
+				<xacro:box_inertia m="0.01" x="0.07" y="0.3" z = "0.09"/>
+		</inertial>
+	</link>
+	<joint name="stereo_camera_joint" type="fixed">
+			<origin rpy="0 0 0" xyz="${chassis_length/2} 0 ${chassis_height/7}"/>
+			<parent link="base_link"/>
+			<child link="stereo_camera"/>
+	</joint>
+	<link name="stereo_camera_optical"/>
+	<joint name="stereo_camera_optical_joint" type="fixed">
+		<origin xyz="0 0 0" rpy="${-pi/2} 0 ${-pi/2}"/>
+		<parent link="stereo_camera"/>
+		<child link="stereo_camera_optical"/>
+	</joint>
+</xacro:if>
 <!-- ............................. ROOF ........................................ -->
 <link name="roof_link">

File: urdf/gazebo.xacro (robot description, xacro)
@@ -31,10 +31,10 @@
 <gazebo reference="imu_frame">
 	<sensor name="my_imu" type="imu">
-    <always_on>true</always_on>
-    <plugin name="my_imu_plugin" filename="libgazebo_ros_imu_sensor.so">
-      <topicName>$(arg robot_namespace)/imu</topicName>
-      <updateRate>5</updateRate>
-      <frameName>imu_frame</frameName>
-    </plugin>
+	<always_on>true</always_on>
+	<plugin name="my_imu_plugin" filename="libgazebo_ros_imu_sensor.so">
+	  <topicName>$(arg robot_namespace)/imu</topicName>
+	  <updateRate>5</updateRate>
+	  <frameName>imu_frame</frameName>
+	</plugin>
   </sensor>
 </gazebo>
@@ -53,5 +53,5 @@
 <!-- ........................... 2D LIDAR PLUGIN ................................... -->
 <xacro:if value="$(arg two_d_lidar_enabled)">
-    <gazebo reference="two_d_lidar">
+	<gazebo reference="two_d_lidar">
 		<gravity>true</gravity>
 		<sensor type="ray" name="two_d_lidar">
@@ -85,5 +85,5 @@
 			</plugin>
 		</sensor>
-    </gazebo>
+	</gazebo>
 </xacro:if>
 <!-- ........................... CAMERA PLUGIN ................................... -->
@@ -127,4 +127,59 @@
 	</gazebo>
 </xacro:if>
-<!--................................................................................. -->
+<!-- ...........................STEREO CAMERA PLUGIN ................................... -->
+<xacro:if value="$(arg stereo_camera_enabled)">
+	<gazebo reference="stereo_camera">
+		<sensor type="multicamera" name="stereo_camera">
+			<update_rate>30.0</update_rate>
+			<camera name="left">
+				<horizontal_fov>1.3962634</horizontal_fov>
+				<image>
+				<width>800</width>
+				<height>800</height>
+				<format>R8G8B8</format>
+				</image>
+				<clip>
+				<near>0.3</near>
+				<far>20</far>
+				</clip>
+				<noise>
+				<type>gaussian</type>
+				<mean>0.0</mean>
+				<stddev>0.007</stddev>
+				</noise>
+			</camera>
+			<camera name="right">
+				<pose>0 -0.07 0 0 0 0</pose>
+				<horizontal_fov>1.3962634</horizontal_fov>
+				<image>
+				<width>800</width>
+				<height>800</height>
+				<format>R8G8B8</format>
+				</image>
+				<clip>
+				<near>0.3</near>
+				<far>20</far>
+				</clip>
+				<noise>
+				<type>gaussian</type>
+				<mean>0.0</mean>
+				<stddev>0.007</stddev>
+				</noise>
+			</camera>
+			<plugin name="stereo_camera_controller" filename="libgazebo_ros_multicamera.so">
+				<alwaysOn>true</alwaysOn>
+				<updateRate>0.0</updateRate>
+				<cameraName>stereo_camera</cameraName>
+				<frameName>stereo_camera_optical</frameName>
+				<hackBaseline>0.07</hackBaseline>
+				<distortionK1>0.0</distortionK1>
+				<distortionK2>0.0</distortionK2>
+				<distortionK3>0.0</distortionK3>
+				<distortionT1>0.0</distortionT1>
+				<distortionT2>0.0</distortionT2>
+				<robotNamespace>$(arg robot_namespace)</robotNamespace>
+			</plugin>
+		</sensor>
+  </gazebo>
+</xacro:if>
 </robot>

Commit message: Added base_footprint tf

File: urdf/bcr_bot.xacro (robot description, xacro)
@@ -42,5 +42,11 @@
     <xacro:include filename="$(find bcr_bot)/urdf/gazebo.xacro"/>
     <!-- ................................ BASE LINK .................................. -->
+    <link name="base_footprint"/>
     <link name="base_link"/>
+    <joint name="base_joint" type="fixed">
+        <parent link="base_footprint"/>
+        <child link="base_link"/>
+        <origin xyz="0.0 0 ${chassis_height/2 + traction_wheel_radius}" rpy="0 0 0.0" />
+    </joint>
     <link name="chassis_link">
         <collision>

File: urdf/gazebo.xacro (robot description, xacro)
@@ -14,5 +14,5 @@
             <wheelSeparation>${traction_track_width+traction_wheel_width-0.01}</wheelSeparation>
             <wheelDiameter>${2*traction_wheel_radius+0.01}</wheelDiameter>
-            <robotBaseFrame>base_link</robotBaseFrame>
+            <robotBaseFrame>base_footprint</robotBaseFrame>
             <wheelTorque>${traction_max_wheel_torque}</wheelTorque>
             <commandTopic>cmd_vel</commandTopic>
@@ -45,5 +45,5 @@
             <alwaysOn>true</alwaysOn>
             <updateRate>30.0</updateRate>
-            <bodyName>base_link</bodyName>
+            <bodyName>base_footprint</bodyName>
             <topicName>ground_truth_pose</topicName>
             <gaussianNoise>0.00</gaussianNoise>

Commit message: Update repo

File: urdf/bcr_bot.xacro (robot description, xacro)
@@ -22,7 +22,7 @@
     <xacro:property name="two_d_lidar_sample_size" value="361"/>
     <xacro:property name="two_d_lidar_min_angle" value="0"/>
-    <xacro:property name="two_d_lidar_max_angle" value="360"/>
+    <xacro:property name="two_d_lidar_max_angle" value="180"/>
     <xacro:property name="two_d_lidar_min_range" value="0.55"/>
-    <xacro:property name="two_d_lidar_max_range" value="16"/>
+    <xacro:property name="two_d_lidar_max_range" value="30"/>
     <xacro:property name="camera_baseline" value="0.06"/>
     <xacro:property name="camera_height" value="0.10"/>
@@ -54,11 +54,11 @@
     </xacro:if>
     <!-- ................................ BASE LINK .................................. -->
-    <link name="base_footprint"/>
+    <!-- <link name="base_footprint"/> -->
     <link name="base_link"/>
-    <joint name="base_joint" type="fixed">
+    <!-- <joint name="base_joint" type="fixed">
         <parent link="base_footprint"/>
         <child link="base_link"/>
         <origin xyz="0.0 0 ${chassis_height/2 + traction_wheel_radius}" rpy="0 0 0.0" />
-    </joint>
+    </joint> -->
     <link name="chassis_link">
         <collision>
@@ -116,5 +116,5 @@
             <parent link="base_link"/>
             <child link="two_d_lidar"/>
-            <origin xyz="0.0 0 0.08" rpy="0 0 0" />
+            <origin xyz="0.0 0 0.08" rpy="0 0 -1.57" />
         </joint>
         <gazebo reference="two_d_lidar">

File: urdf/ign.xacro (robot description, xacro)
@@ -23,5 +23,5 @@
             </xacro:if>
             <frame_id>odom</frame_id>
-            <child_frame_id>base_footprint</child_frame_id>
+            <child_frame_id>base_link</child_frame_id>
         </plugin>
     </gazebo>
@@ -32,5 +32,5 @@
             name="ignition::gazebo::systems::OdometryPublisher">
             <odom_frame>odom</odom_frame>
-            <robot_base_frame>base_footprint</robot_base_frame>
+            <robot_base_frame>base_link</robot_base_frame>
             <odom_topic>$(arg wheel_odom_topic)</odom_topic>
             <tf_topic>/tf</tf_topic>
