Commit message: Add runtime converter for urdf to mjcf model

File: urdf/bcr_bot.xacro (robot description, xacro)
@@ -40,5 +40,12 @@
     <xacro:arg name="sim_gz" default="false" />
     <xacro:arg name="sim_mujoco" default="false" />
+    <xacro:arg name="runtime_mjcf" default="false" />
     <xacro:arg name="odometry_source" default="world" />
+    <!-- D415 DAE coordinates are in centimetres. The MuJoCo converter's
+         DAE-to-OBJ path does not apply the declared unit conversion. -->
+    <xacro:property name="d415_mesh_scale" value="1 1 1"/>
+    <xacro:if value="$(arg runtime_mjcf)">
+        <xacro:property name="d415_mesh_scale" value="0.01 0.01 0.01"/>
+    </xacro:if>
     <xacro:property name="odometry_source" value="$(arg odometry_source)"/>
     <!-- ............................... LOAD MACROS ................................. -->
@@ -73,9 +80,18 @@
         </collision>
         <visual>
-            <origin xyz="0 0 -0.205" rpy="0 0 0" />
+            <origin xyz="0 0 -0.205" rpy="0 0 0"/>
             <geometry>
                 <mesh filename="file://$(find bcr_bot)/meshes/bcr_bot_mesh.dae" scale="1 1 1"/>
             </geometry>
         </visual>
+        <!-- The released converter derives collisions from URDF visuals.
+             Transparent primitive proxies preserve the simple collision shapes. -->
+        <xacro:if value="$(arg runtime_mjcf)">
+            <visual>
+                <origin xyz="0 0 -0.05"/>
+                <geometry><box size="${chassis_length} ${chassis_width} ${chassis_height}"/></geometry>
+                <material name="runtime_collision_proxy"><color rgba="0 0 0 0"/></material>
+            </visual>
+        </xacro:if>
         <inertial>
             <mass value="${chassis_mass}" />
@@ -105,5 +121,5 @@
             </collision>
             <visual>
-                <origin xyz="0 0 0" rpy="0 0 0" />
+                <origin xyz="0 0 0" rpy="0 0 0"/>
                 <geometry>
                     <cylinder length="0.06" radius="0.075"/>
@@ -144,10 +160,16 @@
             </collision>
             <visual>
-                <origin xyz="0 0 0" rpy="0 0 0" />
-                <geometry>
-                    <mesh filename="file://$(find bcr_bot)/meshes/kinect/d415.dae"/>
+                <origin xyz="0 0 0" rpy="0 0 0"/>
+                <geometry>
+                    <mesh filename="file://$(find bcr_bot)/meshes/kinect/d415.dae" scale="${d415_mesh_scale}"/>
                 </geometry>
                 <material name="black"/>
             </visual>
+            <xacro:if value="$(arg runtime_mjcf)">
+                <visual>
+                    <geometry><box size="0.07 0.3 0.09"/></geometry>
+                    <material name="runtime_collision_proxy"><color rgba="0 0 0 0"/></material>
+                </visual>
+            </xacro:if>
             <inertial>
                 <mass value="0.01"/>
@@ -178,10 +200,16 @@
             </collision>
             <visual>
-                <origin xyz="0 0 0" rpy="0 0 0" />
-                <geometry>
-                    <mesh filename="file://$(find bcr_bot)/meshes/kinect/d415.dae"/>
+                <origin xyz="0 0 0" rpy="0 0 0"/>
+                <geometry>
+                    <mesh filename="file://$(find bcr_bot)/meshes/kinect/d415.dae" scale="${d415_mesh_scale}"/>
                 </geometry>
                 <material name="black"/>
             </visual>
+            <xacro:if value="$(arg runtime_mjcf)">
+                <visual>
+                    <geometry><box size="0.07 0.3 0.09"/></geometry>
+                    <material name="runtime_collision_proxy"><color rgba="0 0 0 0"/></material>
+                </visual>
+            </xacro:if>
             <inertial>
                 <mass value="0.01"/>
@@ -200,7 +228,21 @@
             <child link="stereo_camera_optical"/>
         </joint>
+        <xacro:if value="$(arg runtime_mjcf)">
+            <link name="stereo_camera_right_optical"/>
+            <joint name="stereo_camera_right_optical_joint" type="fixed">
+                <origin xyz="0 -0.12 0" rpy="${-pi/2} 0 ${-pi/2}"/>
+                <parent link="stereo_camera"/>
+                <child link="stereo_camera_right_optical"/>
+            </joint>
+        </xacro:if>
     </xacro:if>
     <!-- ............................. ROOF ........................................ -->
     <link name="roof_link">
+        <xacro:if value="$(arg runtime_mjcf)">
+            <visual>
+                <geometry><box size="${chassis_length} ${chassis_width} 0.015"/></geometry>
+                <material name="runtime_collision_proxy"><color rgba="0 0 0 0"/></material>
+            </visual>
+        </xacro:if>
         <collision>
             <origin xyz="0 0 0" rpy="0 0 0" />

File: urdf/macros.xacro (robot description, xacro)
@@ -14,4 +14,10 @@
     <xacro:macro name="trolley_wheel" params="cardinality dexterity origin_x origin_y origin_z">
         <link name="${cardinality}_${dexterity}_wheel">
+            <xacro:if value="$(arg runtime_mjcf)">
+                <visual>
+                    <geometry><sphere radius="${trolley_wheel_radius}"/></geometry>
+                    <material name="runtime_collision_proxy"><color rgba="0 0 0 0"/></material>
+                </visual>
+            </xacro:if>
             <collision>
                 <origin xyz="0 0 0" rpy="0 ${pi/2} ${pi/2}" />
@@ -39,4 +45,11 @@
     <xacro:macro name="traction_wheel" params="cardinality dexterity origin_x origin_y origin_z">
         <link name="${cardinality}_${dexterity}_wheel">
+            <xacro:if value="$(arg runtime_mjcf)">
+                <visual>
+                    <origin xyz="0 0 0" rpy="0 ${pi/2} ${pi/2}"/>
+                    <geometry><cylinder length="${traction_wheel_width}" radius="${traction_wheel_radius}"/></geometry>
+                    <material name="runtime_collision_proxy"><color rgba="0 0 0 0"/></material>
+                </visual>
+            </xacro:if>
             <collision>
                 <origin xyz="0 0 0" rpy="0 ${pi/2} ${pi/2}" />

File: urdf/mujoco_ros2_control.xacro (robot description, xacro)
@@ -4,5 +4,10 @@
         <hardware>
             <plugin>mujoco_ros2_control/MujocoSystemInterface</plugin>
-            <param name="mujoco_model">$(find bcr_bot)/mjcf/small_warehouse.xml</param>
+            <xacro:if value="$(arg runtime_mjcf)">
+                <param name="mujoco_model_topic">/mujoco_robot_description</param>
+            </xacro:if>
+            <xacro:unless value="$(arg runtime_mjcf)">
+                <param name="mujoco_model">$(find bcr_bot)/mjcf/small_warehouse_bcr_bot.xml</param>
+            </xacro:unless>
             <param name="headless">false</param>
             <param name="camera_publish_rate">15.0</param>
@@ -63,3 +68,45 @@
         </sensor>
     </ros2_control>
+    <xacro:if value="$(arg runtime_mjcf)">
+        <mujoco_inputs>
+            <raw_inputs>
+                <compiler fusestatic="true"/>
+                <option timestep="0.002" gravity="0 0 -9.81"/>
+                <default>
+                    <default class="collision">
+                        <geom type="mesh" group="3" rgba="0 0 0 0"/>
+                    </default>
+                    <default class="visual">
+                        <geom type="mesh" contype="0" conaffinity="0" density="0" group="2"/>
+                    </default>
+                </default>
+                <include file="$(find bcr_bot)/mjcf/small_warehouse.xml"/>
+                <actuator>
+                    <velocity name="middle_left_wheel_joint"
+                              joint="middle_left_wheel_joint" kv="100"
+                              forcelimited="true" forcerange="-20000 20000"/>
+                    <velocity name="middle_right_wheel_joint"
+                              joint="middle_right_wheel_joint" kv="100"
+                              forcelimited="true" forcerange="-20000 20000"/>
+                </actuator>
+                <sensor>
+                    <framequat name="imu_quat" objtype="site" objname="imu_frame"/>
+                    <gyro name="imu_gyro" site="imu_frame"/>
+                    <accelerometer name="imu_accel" site="imu_frame"/>
+                    <rangefinder name="two_d_lidar" site="two_d_lidar_ray"/>
+                </sensor>
+            </raw_inputs>
+            <processed_inputs>
+                <camera site="kinect_camera_optical" name="kinect_camera_sensor"
+                        fovy="46.8264488927" mode="fixed" resolution="640 480"/>
+                <camera site="stereo_camera_optical" name="stereo_camera_left"
+                        fovy="64.365484" mode="fixed" resolution="640 480"/>
+                <camera site="stereo_camera_right_optical" name="stereo_camera_right"
+                        fovy="64.365484" mode="fixed" resolution="640 480"/>
+                <lidar ref_site="two_d_lidar" sensor_name="two_d_lidar_ray"
+                       min_angle="0.0" max_angle="6.2831853072"
+                       angle_increment="0.0174532925"/>
+            </processed_inputs>
+        </mujoco_inputs>
+    </xacro:if>
 </robot>

Commit message: Fix runtime MJCF mass, collision geometry, and wheel contacts

File: urdf/bcr_bot.xacro (robot description, xacro)
@@ -65,5 +65,16 @@
     </xacro:if>
     <!-- ................................ BASE LINK .................................. -->
-    <link name="base_footprint"/>
+    <link name="base_footprint">
+        <!-- A tiny runtime-only inertial makes the URDF-to-MJCF converter retain
+             the combined inertial of links merged by fusestatic. Without it,
+             MuJoCo re-infers the fused base mass from collision geometry. -->
+        <xacro:if value="$(arg runtime_mjcf)">
+            <inertial>
+                <mass value="0.000001"/>
+                <inertia ixx="0.000001" ixy="0" ixz="0"
+                         iyy="0.000001" iyz="0" izz="0.000001"/>
+            </inertial>
+        </xacro:if>
+    </link>
     <link name="base_link"/>
     <joint name="base_joint" type="fixed">

File: urdf/macros.xacro (robot description, xacro)
@@ -16,5 +16,8 @@
             <xacro:if value="$(arg runtime_mjcf)">
                 <visual>
-                    <geometry><sphere radius="${trolley_wheel_radius}"/></geometry>
+                    <geometry>
+                        <mesh filename="file://$(find bcr_bot)/meshes/mujoco_runtime/trolley_wheel.obj"
+                              scale="${trolley_wheel_radius} ${trolley_wheel_radius} ${trolley_wheel_radius}"/>
+                    </geometry>
                     <material name="runtime_collision_proxy"><color rgba="0 0 0 0"/></material>
                 </visual>
@@ -23,5 +26,11 @@
                 <origin xyz="0 0 0" rpy="0 ${pi/2} ${pi/2}" />
                 <geometry>
-                    <sphere radius="${trolley_wheel_radius}"/>
+                    <xacro:if value="$(arg runtime_mjcf)">
+                        <mesh filename="file://$(find bcr_bot)/meshes/mujoco_runtime/trolley_wheel.obj"
+                              scale="${trolley_wheel_radius} ${trolley_wheel_radius} ${trolley_wheel_radius}"/>
+                    </xacro:if>
+                    <xacro:unless value="$(arg runtime_mjcf)">
+                        <sphere radius="${trolley_wheel_radius}"/>
+                    </xacro:unless>
                 </geometry>
             </collision>
@@ -48,5 +57,8 @@
                 <visual>
                     <origin xyz="0 0 0" rpy="0 ${pi/2} ${pi/2}"/>
-                    <geometry><cylinder length="${traction_wheel_width}" radius="${traction_wheel_radius}"/></geometry>
+                    <geometry>
+                        <mesh filename="file://$(find bcr_bot)/meshes/mujoco_runtime/traction_wheel.obj"
+                              scale="${traction_wheel_radius} ${traction_wheel_radius} ${traction_wheel_width}"/>
+                    </geometry>
                     <material name="runtime_collision_proxy"><color rgba="0 0 0 0"/></material>
                 </visual>
@@ -55,5 +67,11 @@
                 <origin xyz="0 0 0" rpy="0 ${pi/2} ${pi/2}" />
                 <geometry>
-                    <cylinder length="${traction_wheel_width}" radius="${traction_wheel_radius}"/>
+                    <xacro:if value="$(arg runtime_mjcf)">
+                        <mesh filename="file://$(find bcr_bot)/meshes/mujoco_runtime/traction_wheel.obj"
+                              scale="${traction_wheel_radius} ${traction_wheel_radius} ${traction_wheel_width}"/>
+                    </xacro:if>
+                    <xacro:unless value="$(arg runtime_mjcf)">
+                        <cylinder length="${traction_wheel_width}" radius="${traction_wheel_radius}"/>
+                    </xacro:unless>
                 </geometry>
                 <self_collide>false</self_collide>

File: urdf/mujoco_ros2_control.xacro (robot description, xacro)
@@ -98,4 +98,14 @@
             </raw_inputs>
             <processed_inputs>
+                <!-- Match the contact behavior used by the hand-authored MJCF. -->
+                <modify_element type="body" name="base_footprint"
+                                pos="0 0 0.022"/>
+                <modify_element type="geom" mesh="trolley_wheel" class="collision"
+                                friction="0 0 0" priority="1" condim="1"/>
+                <modify_element type="geom" mesh="traction_wheel" class="collision"
+                                friction="5 0 0"/>
+                <!-- Trolley wheel meshes are collision-only proxies. -->
+                <modify_element type="geom" mesh="trolley_wheel" class="visual"
+                                rgba="0 0 0 0"/>
                 <camera site="kinect_camera_optical" name="kinect_camera_sensor"
                         fovy="46.8264488927" mode="fixed" resolution="640 480"/>
